File: pcb/duckypad.brd (EAGLE design)
At the start: 110 x 96 mm, 87 parts, among them IC2 REG1117, SW21 EC12E_SW, SW22 EC12E_SW, U2 USBC_16P, U3 ESP32-S3FN8

Commit message: working on pcb
Parts:
- removed E1: ANTENNA, esp32-thing-temp:TRACE_ANTENNA_2.4GHZ_25.7MM_TUNED
- removed E2: ANTENNA-GROUNDEDTRACE-15.2MM, SparkFun-RF:TRACE_ANTENNA_2.4GHZ_15.2MM
- added C3, C8: 12pF, clock:0805
- added C4: 1uF, clock:0805
- added JP2: (no value), adafruit_changed:1X03-CLEANBIG
- added R2: 10K, joyAnalog:0805
- added R3, R4: 5.1K, joyAnalog:0805
- added SW1, SW2: SPST_TACT-EVQQ2, adafruit_changed:EVQ-Q2
- added SW3: 324_SW324_SWITCH_FOOT_HOLE, 3pos_slide_switch:342_SWICH_FOOT_HOLE
- added U1: USBC_16P, my_usbc_16p:USBC_16P_FOOT
- added Y1: 16MHz_12pF, SparkFun-Clocks:CRYSTAL-SMD-3.2X2.5MM
- C1, C10, C11, C12, C13, C14, C15, C16, C17, C18, C19, C2, C20, C21, C22, C23, C24, C25, C29, C9: device clock:0805@1 -> clock:0805
- moved C1 8.51 mm to (66.8, 65.2), flipped to the bottom, turned to 0 degrees
- moved C2 4.98 mm to (69.2, 61.2), flipped to the bottom
- moved X1 4.60 mm to (60.4, 63.4), turned to 270 degrees
- moved U3 4.51 mm to (63.0, 54.9)
- moved SD1 1.00 mm to (81.2, 44.3)
- moved U$2 0.27 mm to (72.8, 31.0)
Connections:
- new net N$24: C8.1, U3.54, Y1.1
- new net N$25: C3.1, U3.53, Y1.3
- new net N$26: U3.1, X1.3
- new net N$27: C4.1, R2.2, SW3.P$2, SW3.P$3, U3.4
- new net N$28: R3.1, U1.B5
- new net N$30: R4.1, U1.A5
- new net N$32: C29.2, IC2.3, JP2.2
- net +3V3: now also R2.1
- net GND: now also C3.2, C4.2, C8.2, R3.2, R4.2, SW3.P$1, SW3.P$4, U1.A1B12, U1.B11A12, U1.P$13, U1.P$14, U1.P$15, U1.P$16, X1.1, X1.2, Y1.2, Y1.4
- net N$1: now also JP2.1, U1.A4B9, U1.B4A9; no longer C29.2, IC2.3
- net USB_DN: now also U1.A7, U1.B7
- net USB_DP: now also U1.A6, U1.B6
Other:
- board text added: "bluetooth keyboard? battery charging facility? rotary encoder RC filter free up JTAG pins, leave to last ADC2 can not be used while wifi is on watch out for strapping pins, maybe wire them up to one of the keys? GPIO3 must have pull resistor, pull to high to free up JTAG pins? SPI2, look at table 5e two USB C sockets, one for data one for charging the battery bank"
- board text removed: "bluetooth keyboard? battery charging facility? rotary encoder RC filter free up JTAG pins, leave to last ADC2 can not be used while wifi is on watch out for strapping pins, maybe wire them up to one of the keys? GPIO3 must have pull resistor, pull to high to free up JTAG pins? SPI2, look at table 5e"

Commit message: working on pcb
Parts:
- added U$18: PINHD1X2, adafruit_changed:1X02
- moved X1 15.9 mm to (63.8, 47.9), turned to 90 degrees
- moved C8 15.1 mm to (67.6, 50.9), turned to 180 degrees
- moved C3 14.9 mm to (70.2, 53.8), turned to 270 degrees
- moved Y1 12.4 mm to (67.6, 53.8), turned to 90 degrees
- moved U3 2.19 mm to (60.8, 55.2), turned to 90 degrees
- moved C2 2.17 mm to (70.0, 63.2)
Connections:
- new net N$34: U$18.2, U3.50
- new net N$35: U$18.1, U3.49
- net USB_DN: now also U3.25
- net USB_DP: now also U3.26

Commit message: working on pcb
Parts:
- moved SD1 0.68 mm to (81.0, 45.0)
- moved SW3 0.22 mm to (88.5, 75.5)
- moved U2 0.20 mm to (68.0, 92.0)
- moved U1 0.16 mm to (86.0, 20.0)
Routing:
- added copper zone on layer 16, net GND
- removed copper zone on layer 16, net +3V3

Commit message: working on pcb
Parts:
- added C26, C28, C30, C6: 100nF, clock:0805
- added C5, C7: 1uF, clock:0805
- moved R2 154.5 mm to (85.2, 75.3), flipped to the bottom, turned to 270 degrees
- moved C4 154.2 mm to (82.9, 75.3), flipped to the bottom, turned to 270 degrees
- moved R3 130.4 mm to (85.6, 26.5), flipped to the bottom
- moved R4 125.6 mm to (85.1, 13.5), flipped to the bottom, turned to 180 degrees
- moved X1 2.88 mm to (66.4, 48.9), turned to 180 degrees
- moved U$18 0.89 mm to (68.7, 57.4)
Connections:
- net +3V3: now also C26.2, C28.2, C30.2, C5.2, C6.2, C7.2
- net GND: now also C26.1, C28.1, C30.1, C5.1, C6.1, C7.1
Routing:
- net +3V3: track 0.00 -> 11.5 mm
- net N$25: track 0.00 -> 6.80 mm
- net N$34: track 0.00 -> 6.68 mm
- net N$24: track 0.00 -> 4.49 mm
- net N$35: track 0.00 -> 3.97 mm

Commit message: working on pcb
Parts:
- added C31, C33: 4.7uF, clock:0805
- added C35: 22pF, clock:0805
- added D1: BAT20J, SparkFun-DiscreteSemi:SOD-323
- added L1: 6.8uH, basicBoard:0805
- added R10: 13.3K, joyAnalog:0805
- added R7: 117K, joyAnalog:0805
- added U$19: V_REG_TPS61040SMD, SparkFun-Retired:SOT23-5
Connections:
- new net 12V: C31.2, C35.2, D1.C, R7.1
- new net N$36: D1.A, L1.2, U$19.1
- new net N$39: C35.1, R10.1, R7.2, U$19.3
- net +3V3: now also C33.2, L1.1, U$19.4, U$19.5
- net GND: now also C31.1, C33.1, R10.2, U$19.2

Commit message: working on pcb
Parts:
- removed JP1: (no value), pinhead:1X05
- added C32, C37: 100nF, clock:0805
- added C34: 2.2uF, clock:0805
- added C36: 4.7uF, clock:0805
- added R6: 560K, joyAnalog:0805
- R10: value 13.3K -> 62K
- R7: value 117K -> 560K
- moved C31 179.3 mm to (66.8, 67.6)
- moved R10 176.5 mm to (58.7, 73.2)
- moved R7 171.3 mm to (63.9, 64.3)
- moved L1 171.2 mm to (67.7, 69.5)
- moved C35 167.9 mm to (60.6, 66.4)
- moved C33 167.9 mm to (62.5, 73.0)
- moved D1 167.6 mm to (58.5, 69.8), turned to 270 degrees
- moved U$19 163.4 mm to (63.1, 69.0)
- moved C27 48.4 mm to (75.7, 77.3), turned to 270 degrees
- moved C9 12.0 mm to (62.6, 79.8), turned to 270 degrees
- moved C10 8.07 mm to (57.3, 80.0)
- moved IC2 3.00 mm to (68.7, 78.6), turned to 270 degrees
Connections:
- removed net N$14: SD1.9
- removed net SD_CS: SD1.2
- removed net SPI_MOSI: SD1.3
- removed net UART1_TX: JP1.3
- new net VSS: SD1.6
- net +3V3: now also C36.2, C37.2, U$2.4; no longer JP1.4
- net 12V: now also C32.2, U$2.11, U$2.2
- net GND: now also C32.1, C34.1, C36.1, C37.1, R6.1, U$2.1, U$2.12, U$2.31, U$2.32; no longer JP1.5, SD1.6
- net N$10: now also R6.2, U$2.5; no longer SD1.7
- net N$8: now also C34.2, U$2.3; no longer SD1.5
Other:
- board text removed: "DFU"

Commit message: working on pcb
Parts:
- added R8: 5.1K, joyAnalog:0805
Connections:
- new net N$14: R8.1, U$2.7
- net GND: now also R8.2

Commit message: working on pcb
Parts:
- moved R1 33.1 mm to (66.4, 93.6), flipped to the bottom
- moved R9 25.3 mm to (69.4, 93.6), flipped to the bottom
- moved R3 13.8 mm to (83.4, 13.0)
- moved R4 13.6 mm to (83.4, 26.9), turned to 0 degrees
Routing:
- net N$1: track 0.00 -> 7.56 mm
Changed lines of the file:
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@@
 <element name="U$16" library="3pos_slide_switch_centered" package="M2_SCREW_FOOT" value="M2_SCREW_DEV" x="38.5" y="38.5" smashed="yes"/>
 <element name="U2" library="my_usbc_16p" package="USBC_16P_FOOT" value="USBC_16P" x="68" y="92" smashed="yes" rot="R180"/>
-<element name="R1" library="joyAnalog" package="0805" value="5.1K" x="99.2" y="98.567" smashed="yes" rot="R90">
-<attribute name="NAME" x="99.5683" y="100.472" size="0.8128" layer="25" rot="R90"/>
-</element>
-<element name="R9" library="joyAnalog" package="0805" value="5.1K" x="94.168" y="98.567" smashed="yes" rot="R90">
-<attribute name="NAME" x="94.4347" y="100.4466" size="0.8128" layer="25" rot="R90"/>
+<element name="R1" library="joyAnalog" package="0805" value="5.1K" x="66.434" y="93.614" smashed="yes" rot="MR90">
+<attribute name="NAME" x="66.0657" y="95.519" size="0.8128" layer="26" rot="MR90"/>
+</element>
+<element name="R9" library="joyAnalog" package="0805" value="5.1K" x="69.403" y="93.614" smashed="yes" rot="MR90">
+<attribute name="NAME" x="69.1363" y="95.4936" size="0.8128" layer="26" rot="MR90"/>
 </element>
 <element name="C29" library="clock" package="0805" value="100nF" x="72.517" y="85.0138" smashed="yes" rot="R90">
@@
 </element>
 <element name="SW3" library="3pos_slide_switch" package="342_SWICH_FOOT_HOLE" value="324_SW324_SWITCH_FOOT_HOLE" x="88.5" y="75.5" smashed="yes" rot="MR270"/>
-<element name="R3" library="joyAnalog" package="0805" value="5.1K" x="85.598" y="26.543" smashed="yes" rot="MR0">
-<attribute name="NAME" x="86.36" y="27.3685" size="0.8128" layer="26" rot="MR0"/>
-</element>
-<element name="R4" library="joyAnalog" package="0805" value="5.1K" x="85.09" y="13.462" smashed="yes" rot="MR180">
-<attribute name="NAME" x="84.328" y="12.6365" size="0.8128" layer="26" rot="MR180"/>
+<element name="R3" library="joyAnalog" package="0805" value="5.1K" x="83.439" y="12.954" smashed="yes" rot="MR0">
+<attribute name="NAME" x="84.201" y="13.7795" size="0.8128" layer="26" rot="MR0"/>
+</element>
+<element name="R4" library="joyAnalog" package="0805" value="5.1K" x="83.439" y="26.924" smashed="yes" rot="MR0">
+<attribute name="NAME" x="84.201" y="27.7495" size="0.8128" layer="26" rot="MR0"/>
 </element>
 <element name="U$18" library="adafruit_changed" package="1X02" value="PINHD1X2" x="68.707" y="57.404" smashed="yes" rot="MR180"/>
@@
 <wire x1="66.689" y1="55.023" x2="68.439" y2="52.673" width="0" layer="19" extent="16-16"/>
 <wire x1="60.833" y1="55.245" x2="66.689" y2="55.023" width="0" layer="19" extent="16-16"/>
-<wire x1="94.168" y1="99.467" x2="89.325" y2="77.55" width="0" layer="19" extent="1-16"/>
 </signal>
 <signal name="+3V3">
@@
 <contactref element="R1" pad="1"/>
 <contactref element="U2" pad="B5"/>
-<wire x1="66.25" y1="88.1525" x2="99.2" y2="97.667" width="0" layer="19" extent="1-1"/>
+<wire x1="66.25" y1="88.1525" x2="66.434" y2="92.714" width="0" layer="19" extent="1-16"/>
 </signal>
 <signal name="N$33">
 <contactref element="R9" pad="1"/>
 <contactref element="U2" pad="A5"/>
-<wire x1="69.25" y1="88.1525" x2="94.168" y2="97.667" width="0" layer="19" extent="1-1"/>
+<wire x1="69.25" y1="88.1525" x2="69.403" y2="92.714" width="0" layer="19" extent="1-16"/>
 </signal>
 <signal name="N$1">
@@
 <contactref element="U1" pad="B4A9"/>
 <contactref element="JP2" pad="1"/>
+<wire x1="82.1525" y1="22.425" x2="83.112" y2="22.425" width="0.4064" layer="16"/>
+<wire x1="83.112" y1="22.425" x2="84.074" y2="21.463" width="0.4064" layer="16"/>
+<wire x1="84.074" y1="21.463" x2="84.074" y2="18.542" width="0.4064" layer="16"/>
+<wire x1="83.107" y1="17.575" x2="82.1525" y2="17.575" width="0.4064" layer="16"/>
+<wire x1="84.074" y1="18.542" x2="83.107" y2="17.575" width="0.4064" layer="16"/>
 <wire x1="65.575" y1="88.1525" x2="70.425" y2="88.1525" width="0" layer="19" extent="1-1"/>
 <wire x1="59.54" y1="90" x2="65.575" y2="88.1525" width="0" layer="19" extent="1-1"/>
 <wire x1="82.1525" y1="22.425" x2="70.425" y2="88.1525" width="0" layer="19" extent="1-16"/>
-<wire x1="82.1525" y1="17.575" x2="82.1525" y2="22.425" width="0" layer="19" extent="16-16"/>
 </signal>
 <signal name="USB_DN">
@@
 <contactref element="R3" pad="1"/>
 <contactref element="U1" pad="B5"/>
-<wire x1="82.1525" y1="18.25" x2="86.498" y2="26.543" width="0" layer="19" extent="16-16"/>
+<wire x1="84.339" y1="12.954" x2="82.1525" y2="18.25" width="0" layer="19" extent="16-16"/>
 </signal>
 <signal name="N$30">
 <contactref element="R4" pad="1"/>
 <contactref element="U1" pad="A5"/>
-<wire x1="84.19" y1="13.462" x2="82.1525" y2="21.25" width="0" layer="19" extent="16-16"/>
+<wire x1="82.1525" y1="21.25" x2="84.339" y2="26.924" width="0" layer="19" extent="16-16"/>
 </signal>
 <signal name="N$32">
