File: pcb/duckypad.brd (EAGLE design)
At the start: 110 x 96 mm, 124 parts, among them IC2 REG1117, SW1 SPST_TACT-EVQQ2, SW2 SPST_TACT-EVQQ2, SW21 EC12E_SW, SW22 EC12E_SW, SW3 324_SW324_SWITCH_FOOT_HOLE, U1 USBC_16P, U2 USBC_16P, U3 ESP32-S3FN8, Y1 16MHz_12pF

Commit message: working on top
Parts:
- moved R9 10.6 mm to (73.6, 83.9), flipped to the top, turned to 270 degrees
- moved R1 8.38 mm to (74.8, 94.1), flipped to the top, turned to 270 degrees
- moved U2 0.13 mm to (68.0, 92.1)
Routing:
- net N$31: track 0.00 -> 13.6 mm
- net N$33: track 0.00 -> 11.7 mm
- net USB_DP: track 342.2 -> 341.6 mm
Other:
- board text added: "rotary encoder RC filter watch out for strapping pins GPIO3 must have pull resistor, pull to high to free up JTAG pins? SPI2, look at table 5e fill in thermals on buttons and UFL connector pullups on rotary encoder? test point on OLED reset?"
- board text removed: "bluetooth keyboard? battery charging facility? rotary encoder RC filter free up JTAG pins, leave to last ADC2 can not be used while wifi is on watch out for strapping pins, maybe wire them up to one of the keys? GPIO3 must have pull resistor, pull to high to free up JTAG pins? SPI2, look at table 5e two USB C sockets, one for data one for charging the battery bank"

Commit message: working on top
Parts:
- added C41, C42, C43, C44, C45: 100nF, clock:0805
- moved R5 19.3 mm to (57.8, 78.5)
- moved C21 1.66 mm to (53.5, 69.8), turned to 90 degrees
- moved C20 1.59 mm to (34.7, 69.8), turned to 90 degrees
- moved C19 1.45 mm to (16.0, 69.8), turned to 90 degrees
- moved C23 0.76 mm to (23.7, 53.0)
- moved C22 0.76 mm to (4.57, 52.8)
- moved C24 0.38 mm to (42.8, 52.8)
Connections:
- net +3V3: now also C41.2, C42.2, C43.2, C44.2, C45.2
- net GND: now also C41.1, C42.1, C43.1, C44.1, C45.1
Routing:
- net +3V3: track 17.8 -> 306.1 mm, vias 0 -> 11
- net N$11: track 161.5 -> 164.6 mm
- net N$29: track 45.3 -> 43.2 mm

Commit message: working on top
Parts:
- moved U$10 127.7 mm to (72.8, 7.00)
- moved SW1 0.50 mm to (80.5, 7.00)
Routing:
- net N$46: track 51.5 -> 49.2 mm
Changed lines of the file:
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@@
 <setting verticaltext="up"/>
 </settings>
-<grid distance="5" unitdist="mil" unit="mil" style="lines" multiple="1" display="yes" altdistance="1" altunitdist="mil" altunit="mil"/>
+<grid distance="5" unitdist="mil" unit="mm" style="lines" multiple="1" display="yes" altdistance="1" altunitdist="mil" altunit="mil"/>
 <layers>
 <layer number="1" name="Top" color="4" fill="1" visible="yes" active="yes"/>
@@
 <element name="U$7" library="duckypad" package="M2_SCREW_FOOT" value="M2_SCREW_DEV" x="19.5" y="19.5" smashed="yes"/>
 <element name="U$9" library="duckypad" package="M2_SCREW_FOOT" value="M2_SCREW_DEV" x="38.5" y="76.5" smashed="yes"/>
-<element name="U$10" library="duckypad" package="M2_SCREW_FOOT" value="M2_SCREW_DEV" x="157" y="103" smashed="yes"/>
+<element name="U$10" library="duckypad" package="M2_SCREW_FOOT" value="M2_SCREW_DEV" x="72.75" y="7" smashed="yes"/>
 <element name="U$11" library="duckypad" package="M2_SCREW_FOOT" value="M2_SCREW_DEV" x="19.5" y="76.5" smashed="yes"/>
 <element name="U$15" library="duckypad" package="M2_SCREW_FOOT" value="M2_SCREW_DEV" x="38.5" y="57.5" smashed="yes"/>
@@
 <attribute name="VALUE" x="70.636" y="58.174" size="0.8128" layer="27" ratio="10" rot="R180"/>
 </element>
-<element name="SW1" library="adafruit_changed" package="EVQ-Q2" value="SPST_TACT-EVQQ2" x="80" y="7" smashed="yes"/>
+<element name="SW1" library="adafruit_changed" package="EVQ-Q2" value="SPST_TACT-EVQQ2" x="80.5" y="7" smashed="yes"/>
 <element name="U1" library="my_usbc_16p" package="USBC_16P_FOOT" value="USBC_16P" x="86" y="20" smashed="yes" rot="MR270"/>
 <element name="JP2" library="adafruit_changed" package="1X03-CLEANBIG" value="" x="57" y="91.35" smashed="yes" rot="MR0">
@@
 <wire x1="54.991" y1="58.801" x2="55.51" y2="58.282" width="0.4064" layer="16"/>
 <wire x1="55.51" y1="58.282" x2="58.674" y2="58.282" width="0.4064" layer="16"/>
-<wire x1="54.991" y1="58.801" x2="45.974" y2="58.801" width="0.4064" layer="1"/>
-<wire x1="45.974" y1="58.801" x2="41.148" y2="53.975" width="0.4064" layer="1"/>
-<via x="41.148" y="53.975" extent="1-16" drill="0.55"/>
-<wire x1="41.148" y1="53.975" x2="41.391" y2="53.732" width="0.4064" layer="16"/>
-<wire x1="41.391" y1="53.732" x2="42.799" y2="53.732" width="0.4064" layer="16"/>
+<wire x1="54.991" y1="58.801" x2="48.006" y2="58.801" width="0.4064" layer="1"/>
+<wire x1="48.006" y1="58.801" x2="43.18" y2="53.975" width="0.4064" layer="1"/>
+<wire x1="43.18" y1="53.975" x2="41.275" y2="53.975" width="0.4064" layer="1"/>
+<via x="41.275" y="53.975" extent="1-16" drill="0.55"/>
+<wire x1="41.275" y1="53.975" x2="41.518" y2="53.732" width="0.4064" layer="16"/>
+<wire x1="41.518" y1="53.732" x2="42.799" y2="53.732" width="0.4064" layer="16"/>
 <wire x1="42.799" y1="53.732" x2="45.382" y2="53.732" width="0.4064" layer="16"/>
 <wire x1="45.382" y1="53.732" x2="45.4" y2="53.75" width="0.4064" layer="16"/>
-<wire x1="41.148" y1="53.975" x2="40.132" y2="54.991" width="0.4064" layer="1"/>
-<wire x1="40.132" y1="54.991" x2="-13.081" y2="54.991" width="0.4064" layer="1"/>
+<wire x1="41.275" y1="53.975" x2="40.259" y2="54.991" width="0.4064" layer="1"/>
+<wire x1="40.259" y1="54.991" x2="-13.081" y2="54.991" width="0.4064" layer="1"/>
 <via x="-13.081" y="54.991" extent="1-16" drill="0.55"/>
 <wire x1="-13.081" y1="54.991" x2="-13.843" y2="54.991" width="0.4064" layer="16"/>
@@
 <wire x1="53.975" y1="33.136" x2="63.246" y2="44.588" width="0" layer="19" extent="16-16"/>
 <wire x1="50.6" y1="33.25" x2="53.975" y2="33.136" width="0" layer="19" extent="16-16"/>
-<wire x1="26.4" y1="53.75" x2="41.148" y2="53.975" width="0" layer="19" extent="16-16"/>
+<wire x1="26.4" y1="53.75" x2="41.275" y2="53.975" width="0" layer="19" extent="16-16"/>
 <wire x1="23.749" y1="52.059" x2="26.4" y2="53.75" width="0" layer="19" extent="16-16"/>
 <wire x1="35.306" y1="33.136" x2="50.6" y2="33.25" width="0" layer="19" extent="16-16"/>
@@
 <wire x1="74.295" y1="11.43" x2="75.057" y2="10.668" width="0.2032" layer="16"/>
 <via x="75.057" y="10.668" extent="1-16" drill="0.55"/>
-<wire x1="75.057" y1="10.668" x2="76.6" y2="9.125" width="0.1524" layer="1"/>
-<wire x1="76.6" y1="9.125" x2="76.6" y2="9" width="0.1524" layer="1"/>
 <wire x1="64.262" y1="11.811" x2="64.643" y2="11.43" width="0.2032" layer="16"/>
-<wire x1="76.6" y1="9" x2="83.4" y2="9" width="0" layer="19" extent="1-1"/>
+<wire x1="77.1" y1="9" x2="83.9" y2="9" width="0" layer="19" extent="1-1"/>
+<wire x1="75.057" y1="10.668" x2="77.1" y2="9" width="0" layer="19" extent="1-1"/>
 </signal>
 <signal name="N$47">

Commit message: working on top
Parts:
- moved C44 35.3 mm to (-2.79, 31.6), turned to 90 degrees
- moved C1 28.6 mm to (96.6, 62.5)
- moved C2 26.8 mm to (96.1, 66.4)
- moved C45 17.5 mm to (-15.4, 15.6), turned to 180 degrees
- moved R6 10.2 mm to (65.9, 32.6), turned to 270 degrees
- moved C6 1.59 mm to (67.6, 58.9)
- moved C5 1.53 mm to (69.3, 58.9)
- moved C13 1.27 mm to (3.81, 14.9)
- moved C15 1.14 mm to (42.9, 15.0)
- moved C40 0.90 mm to (67.6, 32.6), turned to 270 degrees
- moved C30 0.76 mm to (63.2, 42.9)
- moved C37 0.76 mm to (68.8, 37.6)
- moved C32 0.52 mm to (78.5, 32.5)
- moved TP1 0.46 mm to (57.9, 20.1)
- moved C14 0.38 mm to (23.4, 15.0)
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Routing:
- net +3V3: track 306.0 -> 607.7 mm, vias 11 -> 25
- net N$1: track 17.1 -> 308.9 mm, vias 0 -> 2
- net 12V: track 5.96 -> 71.9 mm, vias 0 -> 2
- net N$10: track 0.00 -> 17.4 mm
- net GND: track 0.00 -> 14.7 mm, vias 0 -> 14
- net N$8: track 0.00 -> 5.62 mm
- net N$20: track 162.9 -> 164.8 mm
- net SCLK: track 26.9 -> 28.0 mm
- net MOSI: track 28.6 -> 29.5 mm

Commit message: top routing done
Parts:
- LED_R1C1, LED_R1C2, LED_R1C3, LED_R1C4, LED_R2C1, LED_R2C2, LED_R2C3, LED_R2C4, LED_R3C1, LED_R3C2, LED_R3C3, LED_R3C4, LED_R4C1, LED_R4C2, LED_R4C3, LED_R4C4, LED_R5C1, LED_R5C2, LED_R5C3, LED_R5C4: device lul:REVERSE_MNT -> duckypad:REVERSE_MNT
- moved U$18 62.5 mm to (17.3, 92.3), turned to 180 degrees
- moved C26 2.45 mm to (70.6, 55.5), turned to 270 degrees
- moved C7 2.45 mm to (68.8, 55.5), turned to 270 degrees
- moved SW3 0.13 mm to (88.4, 75.5), turned to 90 degrees
- flipped C10 to the bottom
- flipped C9 to the bottom
Routing:
- net RESET: track 0.00 -> 111.3 mm, vias 0 -> 2
- net SW_R1C3: track 45.2 -> 71.7 mm
- net SW_R1C2: track 72.6 -> 82.1 mm
- net N$46: track 49.2 -> 58.8 mm
- net +3V3: track 607.7 -> 613.6 mm
- net N$3: track 14.4 -> 19.3 mm
- net USB_DP: track 341.6 -> 340.0 mm
- net SW_R3C3: track 27.2 -> 26.2 mm
- net N$1: track 308.9 -> 309.6 mm
- net N$47: track 47.8 -> 48.4 mm
- net GND: vias 14 -> 21

Commit message: finishing touches
Parts:
- removed C1, C10, C2, C9: 100nF, clock:0805
Connections:
- net +3V3: no longer C1.2, C10.2, C2.2, C9.2
- net GND: no longer C1.1, C10.1, C2.1, C9.1
Routing:
- net +3V3: track 613.6 -> 612.0 mm
- net N$5: track 29.7 -> 29.1 mm

Commit message: time for silkscreen
Parts:
- removed TP1: TPTP12R, testpad:TP12R
- added JP1: (no value), adafruit_changed:1X01-CLEANBIG
- moved R2 23.6 mm to (72.4, 55.5), flipped to the bottom, turned to 90 degrees
- moved X1 4.85 mm to (69.9, 59.8)
- moved C44 2.54 mm to (-2.92, 34.2), turned to 270 degrees
- moved C6 1.35 mm to (68.6, 59.8), turned to 0 degrees
- moved C5 1.17 mm to (68.6, 58.0), turned to 0 degrees
- moved C4 1.14 mm to (84.8, 75.2)
- moved C45 0.90 mm to (-14.7, 15.0), turned to 90 degrees
- moved C31 0.25 mm to (59.7, 67.1)
Connections:
- net N$27: now also JP1.1; no longer TP1.TP
Routing:
- net N$26: track 2.45 -> 7.14 mm
- net RESET: track 111.3 -> 116.0 mm
- net N$38: track 39.1 -> 41.7 mm
- net N$37: track 51.4 -> 54.1 mm
- net N$40: track 45.6 -> 47.0 mm
- net N$43: track 22.6 -> 21.4 mm
- net 12V: track 71.6 -> 70.8 mm
- net +3V3: track 612.0 -> 612.7 mm
Other:
- board text removed: "RST"
