File: pcb/duckypad.sch (EAGLE design)
At the start: 159 parts, among them IC2 REG1117, SW1 SPST_TACT-EVQQ2, SW2 SPST_TACT-EVQQ2, SW21 EC12E_SW, SW22 EC12E_SW, SW3 324_SW324_SWITCH_FOOT_HOLE, SW4 324_SW324_SWITCH_FOOT_HOLE, U1 USBC_16P, U2 USBC_16P, U3 ESP32-S3FN8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

Commit message: silkscreen update
Parts:
- removed R19: DNP, joyAnalog:RESISTOR0805-RES
- added JP4: JUMPER-SMT_2_NO_NO-SILK, SparkFun-Jumpers:JUMPER-SMT_2_NO_NO-SILK
Connections:
- net N$41: now also JP4.2; no longer R19.1
- net RESET: now also JP4.1; no longer R19.2
Changed lines of the file:
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@@
 <part name="C28" library="clock" deviceset="CAP" device="0805" value="100nF"/>
 <part name="GND40" library="supply1" library_urn="urn:adsk.eagle:library:371" deviceset="GND" device=""/>
-<part name="GND41" library="supply1" library_urn="urn:adsk.eagle:library:371" deviceset="GND" device=""/>
 <part name="U$19" library="SparkFun-Retired" deviceset="V_REG_TPS61040" device="SMD"/>
 <part name="+3V32" library="supply1" library_urn="urn:adsk.eagle:library:371" deviceset="+3V3" device=""/>
@@
 <part name="R4" library="joyAnalog" deviceset="RESISTOR" device="0805-RES" value="5K1"/>
 <part name="R18" library="joyAnalog" deviceset="RESISTOR" device="0805-RES" value="5K1"/>
-<part name="R19" library="joyAnalog" deviceset="RESISTOR" device="0805-RES" value="DNP"/>
 <part name="JP1" library="SparkFun-Jumpers" deviceset="JUMPER-SMT_2_NO" device="_NO-SILK"/>
 <part name="GND65" library="supply1" deviceset="GND" device=""/>
+<part name="JP4" library="SparkFun-Jumpers" deviceset="JUMPER-SMT_2_NO" device="_NO-SILK"/>
 </parts>
 <sheets>
@@
 <attribute name="VALUE" x="505.46" y="-35.56" size="1.778" layer="96"/>
 </instance>
-<instance part="GND41" gate="1" x="490.22" y="-35.56" smashed="yes">
-<attribute name="VALUE" x="487.68" y="-38.1" size="1.778" layer="96"/>
-</instance>
 <instance part="U$19" gate="G$1" x="190.5" y="-284.48" smashed="yes">
 <attribute name="NAME" x="185.42" y="-274.32" size="1.778" layer="95" rot="MR180"/>
@@
 <attribute name="VALUE" x="-1.27" y="-189.738" size="1.778" layer="96" rot="MR180"/>
 </instance>
-<instance part="R19" gate="G$1" x="342.9" y="-5.08" smashed="yes" rot="MR270">
-<attribute name="NAME" x="341.4014" y="-1.27" size="1.778" layer="95" rot="MR270"/>
-<attribute name="VALUE" x="346.202" y="-1.27" size="1.778" layer="96" rot="MR270"/>
-<attribute name="NAME" x="341.4014" y="-1.27" size="1.778" layer="95" rot="MR270"/>
-<attribute name="VALUE" x="346.202" y="-1.27" size="1.778" layer="96" rot="MR270"/>
-</instance>
 <instance part="JP1" gate="G$1" x="93.98" y="-137.16" smashed="yes">
 <attribute name="NAME" x="91.44" y="-134.62" size="1.778" layer="95" font="vector"/>
-<attribute name="VALUE" x="91.44" y="-139.7" size="1.778" layer="96" font="vector" align="top-left"/>
 </instance>
 <instance part="GND65" gate="1" x="-10.16" y="-193.04" smashed="yes" rot="MR0">
 <attribute name="VALUE" x="-7.62" y="-195.58" size="1.778" layer="96" rot="MR0"/>
+</instance>
+<instance part="JP4" gate="G$1" x="342.9" y="-5.08" smashed="yes" rot="R90">
+<attribute name="NAME" x="340.36" y="-7.62" size="1.778" layer="95" font="vector" rot="R90"/>
 </instance>
 </instances>
@@
 <wire x1="314.96" y1="-10.16" x2="325.12" y2="-10.16" width="0.1524" layer="91"/>
 <junction x="314.96" y="-10.16"/>
-<pinref part="R19" gate="G$1" pin="2"/>
+<pinref part="JP4" gate="G$1" pin="1"/>
 <junction x="342.9" y="-10.16"/>
 </segment>
@@
 <junction x="398.78" y="-38.1"/>
 <wire x1="375.92" y1="0" x2="342.9" y2="0" width="0.1524" layer="91"/>
-<pinref part="R19" gate="G$1" pin="1"/>
-</segment>
-</net>
+<pinref part="JP4" gate="G$1" pin="2"/>
+</segment>
+</net>

Commit message: updated pcb component values
Parts:
- C26, C6: value 100nF -> 1uF
- C5, C7: value 1uF -> 100nF
- R17, R5: value 10K -> 5K1
Changed lines of the file:
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@@
 <part name="U$6" library="supply1" library_urn="urn:adsk.eagle:library:371" deviceset="GND" device=""/>
 <part name="+3V30" library="supply1" library_urn="urn:adsk.eagle:library:371" deviceset="+3V3" device=""/>
-<part name="R5" library="clock" deviceset="RESISTOR" device="0805-RES" value="10K"/>
+<part name="R5" library="clock" deviceset="RESISTOR" device="0805-RES" value="5K1"/>
 <part name="C27" library="clock" deviceset="C-US" device="C1210" value="100uF"/>
 <part name="U$7" library="duckypad" deviceset="M2_SCREW_DEV" device=""/>
@@
 <part name="GND34" library="clock" deviceset="GND" device=""/>
 <part name="GND35" library="supply1" deviceset="GND" device=""/>
-<part name="C5" library="clock" deviceset="CAP" device="0805" value="1uF"/>
-<part name="C6" library="clock" deviceset="CAP" device="0805" value="100nF"/>
+<part name="C5" library="clock" deviceset="CAP" device="0805" value="100nF"/>
+<part name="C6" library="clock" deviceset="CAP" device="0805" value="1uF"/>
 <part name="GND36" library="supply1" library_urn="urn:adsk.eagle:library:371" deviceset="GND" device=""/>
 <part name="GND37" library="supply1" library_urn="urn:adsk.eagle:library:371" deviceset="GND" device=""/>
-<part name="C7" library="clock" deviceset="CAP" device="0805" value="1uF"/>
-<part name="C26" library="clock" deviceset="CAP" device="0805" value="100nF"/>
+<part name="C7" library="clock" deviceset="CAP" device="0805" value="100nF"/>
+<part name="C26" library="clock" deviceset="CAP" device="0805" value="1uF"/>
 <part name="GND38" library="supply1" library_urn="urn:adsk.eagle:library:371" deviceset="GND" device=""/>
 <part name="GND39" library="supply1" library_urn="urn:adsk.eagle:library:371" deviceset="GND" device=""/>
@@
 <part name="L2" library="Discrete" deviceset="L*" device="-4030" value="4.7uH"/>
 <part name="C46" library="clock" deviceset="CAP" device="0805" value="4.7uF"/>
-<part name="R17" library="joyAnalog" deviceset="RESISTOR" device="0805-RES" value="10K"/>
+<part name="R17" library="joyAnalog" deviceset="RESISTOR" device="0805-RES" value="5K1"/>
 <part name="GND62" library="supply1" library_urn="urn:adsk.eagle:library:371" deviceset="GND" device=""/>
 <part name="JP3" library="adafruit_changed" deviceset="PINHD-1X1" device="CB"/>

Commit message: added more labels, removed m2 screw between +- button
Parts:
- removed U$10: M2_SCREW_DEV, duckypad:M2_SCREW_DEV
- SW1, SW2: device adafruit_changed:SPST_TACT-EVQQ2 -> duckypad:SPST_TACT-EVQQ2
Changed lines of the file:
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@@
 <part name="U$7" library="duckypad" deviceset="M2_SCREW_DEV" device=""/>
 <part name="U$9" library="duckypad" deviceset="M2_SCREW_DEV" device=""/>
-<part name="U$10" library="duckypad" deviceset="M2_SCREW_DEV" device=""/>
 <part name="U$11" library="duckypad" deviceset="M2_SCREW_DEV" device=""/>
 <part name="U$15" library="duckypad" deviceset="M2_SCREW_DEV" device=""/>
@@
 <part name="GND12" library="supply1" library_urn="urn:adsk.eagle:library:371" deviceset="GND" device=""/>
 <part name="X1" library="adafruit_changed" deviceset="ANTENNA_U.FL" device=""/>
-<part name="SW1" library="adafruit_changed" deviceset="SPST_TACT" device="-EVQQ2"/>
+<part name="SW1" library="duckypad" deviceset="SPST_TACT" device="-EVQQ2"/>
 <part name="U1" library="my_usbc_16p" deviceset="USBC_16P" device=""/>
 <part name="JP2" library="adafruit_changed" deviceset="PINHD-1X3" device="CB"/>
-<part name="SW2" library="adafruit_changed" deviceset="SPST_TACT" device="-EVQQ2"/>
+<part name="SW2" library="duckypad" deviceset="SPST_TACT" device="-EVQQ2"/>
 <part name="GND13" library="clock" deviceset="GND" device=""/>
 <part name="C8" library="clock" deviceset="CAP" device="0805" value="12pF"/>
@@
 <instance part="U$7" gate="G$1" x="467.36" y="48.26" smashed="yes"/>
 <instance part="U$9" gate="G$1" x="495.3" y="33.02" smashed="yes"/>
-<instance part="U$10" gate="G$1" x="467.36" y="33.02" smashed="yes"/>
 <instance part="U$11" gate="G$1" x="523.24" y="33.02" smashed="yes"/>
 <instance part="U$15" gate="G$1" x="495.3" y="48.26" smashed="yes"/>

Commit message: adjust values
Parts:
- C26, C6: value 1uF -> 4.7uF
- R1, R9: value 5.1K -> 5K1
- R11, R12, R16: value 10K -> 5K1
Changed lines of the file:
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@@
 <part name="U2" library="my_usbc_16p" deviceset="USBC_16P" device=""/>
 <part name="GND6" library="supply1" deviceset="GND" device=""/>
-<part name="R1" library="joyAnalog" deviceset="RESISTOR" device="0805-RES" value="5.1K"/>
-<part name="R9" library="joyAnalog" deviceset="RESISTOR" device="0805-RES" value="5.1K"/>
+<part name="R1" library="joyAnalog" deviceset="RESISTOR" device="0805-RES" value="5K1"/>
+<part name="R9" library="joyAnalog" deviceset="RESISTOR" device="0805-RES" value="5K1"/>
 <part name="C29" library="clock" deviceset="CAP" device="0805" value="4.7uF"/>
 <part name="GND16" library="supply1" library_urn="urn:adsk.eagle:library:371" deviceset="GND" device=""/>
@@
 <part name="GND35" library="supply1" deviceset="GND" device=""/>
 <part name="C5" library="clock" deviceset="CAP" device="0805" value="100nF"/>
-<part name="C6" library="clock" deviceset="CAP" device="0805" value="1uF"/>
+<part name="C6" library="clock" deviceset="CAP" device="0805" value="4.7uF"/>
 <part name="GND36" library="supply1" library_urn="urn:adsk.eagle:library:371" deviceset="GND" device=""/>
 <part name="GND37" library="supply1" library_urn="urn:adsk.eagle:library:371" deviceset="GND" device=""/>
 <part name="C7" library="clock" deviceset="CAP" device="0805" value="100nF"/>
-<part name="C26" library="clock" deviceset="CAP" device="0805" value="1uF"/>
+<part name="C26" library="clock" deviceset="CAP" device="0805" value="4.7uF"/>
 <part name="GND38" library="supply1" library_urn="urn:adsk.eagle:library:371" deviceset="GND" device=""/>
 <part name="GND39" library="supply1" library_urn="urn:adsk.eagle:library:371" deviceset="GND" device=""/>
@@
 <part name="GND50" library="supply1" library_urn="urn:adsk.eagle:library:371" deviceset="GND" device=""/>
 <part name="GND51" library="supply1" library_urn="urn:adsk.eagle:library:371" deviceset="GND" device=""/>
-<part name="R11" library="joyAnalog" deviceset="RESISTOR" device="0805-RES" value="10K"/>
+<part name="R11" library="joyAnalog" deviceset="RESISTOR" device="0805-RES" value="5K1"/>
 <part name="+3V31" library="supply1" library_urn="urn:adsk.eagle:library:371" deviceset="+3V3" device=""/>
 <part name="C38" library="clock" deviceset="CAP" device="0805" value="4.7uF"/>
@@
 <part name="GND52" library="supply1" library_urn="urn:adsk.eagle:library:371" deviceset="GND" device=""/>
 <part name="GND53" library="supply1" library_urn="urn:adsk.eagle:library:371" deviceset="GND" device=""/>
-<part name="R12" library="joyAnalog" deviceset="RESISTOR" device="0805-RES" value="10K"/>
+<part name="R12" library="joyAnalog" deviceset="RESISTOR" device="0805-RES" value="5K1"/>
 <part name="+3V33" library="supply1" library_urn="urn:adsk.eagle:library:371" deviceset="+3V3" device=""/>
 <part name="C40" library="clock" deviceset="CAP" device="0805" value="100nF"/>
@@
 <part name="C10" library="clock" deviceset="CAP" device="0805" value="100nF"/>
 <part name="GND60" library="supply1" library_urn="urn:adsk.eagle:library:371" deviceset="GND" device=""/>
-<part name="R16" library="joyAnalog" deviceset="RESISTOR" device="0805-RES" value="10K"/>
+<part name="R16" library="joyAnalog" deviceset="RESISTOR" device="0805-RES" value="5K1"/>
 <part name="+3V35" library="supply1" library_urn="urn:adsk.eagle:library:371" deviceset="+3V3" device=""/>
 <part name="L2" library="Discrete" deviceset="L*" device="-4030" value="4.7uH"/>

Commit message: fixed SH socket name
Parts:
- renumbered U$3 to SH1
Changed lines of the file:
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@@
 <part name="GND66" library="supply1" library_urn="urn:adsk.eagle:library:371" deviceset="GND" device=""/>
 <part name="R3" library="adafruit_changed" deviceset="R-US_" device="R2010"/>
-<part name="U$3" library="duckypad" deviceset="SH10P" device=""/>
+<part name="SH1" library="duckypad" deviceset="SH10P" device=""/>
 <part name="+3V39" library="supply1" library_urn="urn:adsk.eagle:library:371" deviceset="+3V3" device=""/>
 <part name="GND70" library="supply1" deviceset="GND" device=""/>
@@
 <attribute name="VALUE" x="275.59" y="-153.162" size="1.778" layer="96"/>
 </instance>
-<instance part="U$3" gate="G$1" x="127" y="-215.9" smashed="yes"/>
+<instance part="SH1" gate="G$1" x="127" y="-215.9" smashed="yes"/>
 <instance part="+3V39" gate="G$1" x="147.32" y="-205.74" smashed="yes" rot="MR0">
 <attribute name="VALUE" x="149.86" y="-210.82" size="1.778" layer="96" rot="MR90"/>
@@
 <segment>
 <pinref part="GND70" gate="1" pin="GND"/>
-<pinref part="U$3" gate="G$1" pin="2"/>
+<pinref part="SH1" gate="G$1" pin="2"/>
 <wire x1="104.14" y1="-205.74" x2="124.46" y2="-205.74" width="0.1524" layer="91"/>
 </segment>
 <segment>
-<pinref part="U$3" gate="G$1" pin="12"/>
+<pinref part="SH1" gate="G$1" pin="12"/>
 <pinref part="GND64" gate="1" pin="GND"/>
 <wire x1="124.46" y1="-233.68" x2="119.38" y2="-233.68" width="0.1524" layer="91"/>
-<pinref part="U$3" gate="G$1" pin="11"/>
+<pinref part="SH1" gate="G$1" pin="11"/>
 <wire x1="124.46" y1="-231.14" x2="119.38" y2="-231.14" width="0.1524" layer="91"/>
 <wire x1="119.38" y1="-231.14" x2="119.38" y2="-233.68" width="0.1524" layer="91"/>
@@
 <segment>
 <pinref part="+3V39" gate="G$1" pin="+3V3"/>
-<pinref part="U$3" gate="G$1" pin="3"/>
+<pinref part="SH1" gate="G$1" pin="3"/>
 <wire x1="147.32" y1="-208.28" x2="124.46" y2="-208.28" width="0.1524" layer="91"/>
 </segment>
@@
 <wire x1="398.78" y1="-78.74" x2="368.3" y2="-78.74" width="0.1524" layer="91"/>
 <wire x1="368.3" y1="-78.74" x2="368.3" y2="-210.82" width="0.1524" layer="91"/>
-<pinref part="U$3" gate="G$1" pin="4"/>
+<pinref part="SH1" gate="G$1" pin="4"/>
 <wire x1="124.46" y1="-210.82" x2="368.3" y2="-210.82" width="0.1524" layer="91"/>
 <label x="124.46" y="-210.82" size="1.778" layer="95" rot="R180" xref="yes"/>
@@
 <wire x1="347.98" y1="-78.74" x2="340.36" y2="-78.74" width="0.1524" layer="91"/>
 <wire x1="340.36" y1="-78.74" x2="340.36" y2="-213.36" width="0.1524" layer="91"/>
-<pinref part="U$3" gate="G$1" pin="5"/>
+<pinref part="SH1" gate="G$1" pin="5"/>
 <wire x1="124.46" y1="-213.36" x2="340.36" y2="-213.36" width="0.1524" layer="91"/>
 </segment>
@@
 <wire x1="337.82" y1="-76.2" x2="337.82" y2="-215.9" width="0.1524" layer="91"/>
 <wire x1="337.82" y1="-215.9" x2="124.46" y2="-215.9" width="0.1524" layer="91"/>
-<pinref part="U$3" gate="G$1" pin="6"/>
+<pinref part="SH1" gate="G$1" pin="6"/>
 </segment>
 </net>
@@
 <wire x1="398.78" y1="-81.28" x2="370.84" y2="-81.28" width="0.1524" layer="91"/>
 <wire x1="370.84" y1="-81.28" x2="370.84" y2="-218.44" width="0.1524" layer="91"/>
-<pinref part="U$3" gate="G$1" pin="7"/>
+<pinref part="SH1" gate="G$1" pin="7"/>
 <wire x1="124.46" y1="-218.44" x2="370.84" y2="-218.44" width="0.1524" layer="91"/>
 </segment>
@@
 <wire x1="373.38" y1="-83.82" x2="373.38" y2="-220.98" width="0.1524" layer="91"/>
 <wire x1="373.38" y1="-220.98" x2="124.46" y2="-220.98" width="0.1524" layer="91"/>
-<pinref part="U$3" gate="G$1" pin="8"/>
+<pinref part="SH1" gate="G$1" pin="8"/>
 </segment>
 </net>
@@
 <wire x1="332.74" y1="-68.58" x2="332.74" y2="-223.52" width="0.1524" layer="91"/>
 <wire x1="332.74" y1="-223.52" x2="124.46" y2="-223.52" width="0.1524" layer="91"/>
-<pinref part="U$3" gate="G$1" pin="9"/>
+<pinref part="SH1" gate="G$1" pin="9"/>
 </segment>
 </net>
@@
 <junction x="335.28" y="-71.12"/>
 <wire x1="335.28" y1="-226.06" x2="124.46" y2="-226.06" width="0.1524" layer="91"/>
-<pinref part="U$3" gate="G$1" pin="10"/>
+<pinref part="SH1" gate="G$1" pin="10"/>
 </segment>
 </net>
@@
 <wire x1="99.06" y1="-144.78" x2="96.52" y2="-144.78" width="0.1524" layer="91"/>
 <wire x1="96.52" y1="-144.78" x2="96.52" y2="-154.94" width="0.1524" layer="91"/>
-<pinref part="U$3" gate="G$1" pin="1"/>
+<pinref part="SH1" gate="G$1" pin="1"/>
 <wire x1="96.52" y1="-154.94" x2="96.52" y2="-177.8" width="0.1524" layer="91"/>
 <wire x1="96.52" y1="-177.8" x2="96.52" y2="-203.2" width="0.1524" layer="91"/>

Commit message: preparing for next run
Parts:
- added R19: 5K1, joyAnalog:RESISTOR0805-RES
- added U$3: BUZZ40402, duckypad:BUZZ40402
Connections:
- new net N$37: R19.1, U$3.PLUS
- net GND: now also U$3.MINUS
- net N$70: now also R19.2
Changed lines of the file:
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@@
 <drawing>
 <settings>
-<setting alwaysvectorfont="yes"/>
+<setting alwaysvectorfont="no"/>
 <setting keepoldvectorfont="yes"/>
 <setting verticaltext="up"/>
@@
 <part name="GND65" library="supply1" deviceset="GND" device=""/>
 <part name="JP4" library="SparkFun-Jumpers" deviceset="JUMPER-SMT_2_NO" device="_NO-SILK"/>
+<part name="U$3" library="duckypad" deviceset="BUZZ40402" device=""/>
+<part name="R19" library="joyAnalog" deviceset="RESISTOR" device="0805-RES" value="5K1"/>
+<part name="GND41" library="supply1" deviceset="GND" device=""/>
 </parts>
 <sheets>
@@
 <attribute name="NAME" x="340.36" y="-7.62" size="1.778" layer="95" font="vector" rot="R90"/>
 </instance>
+<instance part="U$3" gate="G$1" x="93.98" y="-220.98" smashed="yes" rot="MR0"/>
+<instance part="R19" gate="G$1" x="119.38" y="-220.98" smashed="yes" rot="MR180">
+<attribute name="NAME" x="118.11" y="-217.3986" size="1.778" layer="95" rot="MR180"/>
+<attribute name="VALUE" x="118.11" y="-215.138" size="1.778" layer="96" rot="MR180"/>
+</instance>
+<instance part="GND41" gate="1" x="71.12" y="-223.52" smashed="yes" rot="MR0">
+<attribute name="VALUE" x="73.66" y="-226.06" size="1.778" layer="96" rot="MR0"/>
+</instance>
 </instances>
 <busses>
@@
 <junction x="-10.16" y="-185.42"/>
 </segment>
+<segment>
+<pinref part="GND41" gate="1" pin="GND"/>
+<pinref part="U$3" gate="G$1" pin="MINUS"/>
+<wire x1="71.12" y1="-220.98" x2="78.74" y2="-220.98" width="0.1524" layer="91"/>
+</segment>
 </net>
 <net name="+3V3" class="0">
@@
 <wire x1="373.38" y1="-220.98" x2="124.46" y2="-220.98" width="0.1524" layer="91"/>
 <pinref part="SH1" gate="G$1" pin="8"/>
+<pinref part="R19" gate="G$1" pin="2"/>
+<junction x="124.46" y="-220.98"/>
 </segment>
 </net>
@@
 </segment>
 </net>
+<net name="N$37" class="0">
+<segment>
+<pinref part="U$3" gate="G$1" pin="PLUS"/>
+<pinref part="R19" gate="G$1" pin="1"/>
+<wire x1="109.22" y1="-220.98" x2="114.3" y2="-220.98" width="0.1524" layer="91"/>
+</segment>
+</net>
