File: pcb/rev1/duckypad.sch (EAGLE design)
At the start: 159 parts, among them IC2 REG1117, SW1 SPST_TACT-EVQQ2, SW2 SPST_TACT-EVQQ2, SW21 EC12E_SW, SW22 EC12E_SW, SW3 324_SW324_SWITCH_FOOT_HOLE, SW4 324_SW324_SWITCH_FOOT_HOLE, U1 USBC_16P, U2 USBC_16P, U3 ESP32-S3FN8, Y1 16MHz_12pF

Commit message: working on new PCB revision
Parts:
- removed D10, D11, D12, D13, D14, D15, D16, D17, D18, D19, D2, D20, D21, D3, D4, D5, D6, D7, D8, D9: 1N4148, duckypad:ADAFRUIT_CHANGED_DIODESOD-123
- removed R19: DNP, joyAnalog:RESISTOR0805-RES
- removed SW4: 324_SW324_SWITCH_FOOT_HOLE, 3pos_slide_switch:324_SW324_SWITCH_FOOT_HOLE
- removed X2: (no value), adafruit_changed:ANTENNA_U.FL
- added C30, C32: 100nF, clock:CAP0805
- added JP5: (no value), pinhead:PINHD-2X3
- C1, C10, C2, C9: value 100nF -> 10nF
- C27: value 100uF -> 47uF
- C29: value 4.7uF -> 10uF
- C31: value 100nF -> 4.7uF
- C34, C38: value 4.7uF -> 2.2uF
- C35: value 12pF -> 22pF
- C4: value 100nF -> 1uF
- C46: value 4.7uF -> 100nF
- D1: value 1N4148 -> (none); device duckypad:ADAFRUIT_CHANGED_DIODESOD-123 -> adafruit_changed:DIODESOD-123
- JP1: value JUMPER-SMT_2_NO_NO-SILK -> (none); device SparkFun-Jumpers:JUMPER-SMT_2_NO_NO-SILK -> adafruit_changed:PINHD-1X1CB
- L2: value 4.7uH -> PRS4018-4R7MT
- R13, R14, R15, R8: value 5K1 -> 10K
- R2: value 62K -> 10K
- R3: value (none) -> 5.1K; device adafruit_changed:R-US_R2010 -> joyAnalog:RESISTOR0805-RES
- R4: value 470 -> 5.1K
- R5: value 10K -> 5.1K
- R6, R7: value 510K -> 560K
- U$3: value SH10P -> PINHD1X2; device duckypad:SH10P -> adafruit_changed:PINHD1X2
Connections:
- removed net AUX_DN: U1.DN1, U1.DN2, U3.XTAL_32K_P
- removed net AUX_DP: U1.DP1, U1.DP2, U3.XTAL_32K_N
- removed net CC_BUSY: R18.1, R4.1, U$3.4, U3.GPIO21
- removed net COL0: SWR1C1.2, SWR2C1.2, SWR3C1.2, SWR4C1.2, SWR5C1.2, U3.MTMS
- removed net COL1: SWR1C2.2, SWR2C2.2, SWR3C2.2, SWR4C2.2, SWR5C2.2, U3.MTDI
- removed net COL2: SWR1C3.2, SWR2C3.2, SWR3C3.2, SWR4C3.2, SWR5C3.2, U3.MTCK
- removed net COL3: SWR1C4.2, SWR2C4.2, SWR3C4.2, SWR4C4.2, SWR5C4.2, U3.GPIO38
- removed net N$45: D3.A, SWR1C2.1
- removed net N$50: D8.A, SWR2C3.1
- removed net N$51: D7.A, SWR2C2.1
- removed net N$52: D6.A, SWR2C1.1
- removed net N$53: D10.A, SWR3C4.1
- removed net N$54: D11.A, SWR3C3.1
- removed net N$55: D12.A, SWR3C2.1
- removed net N$56: D13.A, SWR3C1.1
- removed net N$57: D17.A, SWR4C4.1
- removed net N$58: D16.A, SWR4C3.1
- removed net N$59: D15.A, SWR4C2.1
- removed net N$60: D14.A, SWR4C1.1
- removed net N$61: D18.A, SWR5C4.1
- removed net N$62: D19.A, SWR5C3.1
- removed net N$63: D20.A, SWR5C2.1
- removed net N$64: D21.A, SWR5C1.1
- removed net N$65: SW2.S, SW2.S1, U3.GPIO18
- removed net N$66: C29.2, IC2.VIN, JP1.2, JP2.2, U$3.1, U1.VBUS
- removed net N$67: U$3.5, U3.SPICLK_N
- removed net N$68: U$3.6, U3.SPICLK_P
- removed net N$69: U$3.7, U3.GPIO33
- removed net N$70: U$3.8, U3.GPIO34
- removed net N$71: R3.1, X2.SIGNAL
- removed net N$72: U$3.9, U3.U0RXD
- removed net N$73: JP3.1, U$3.10, U3.U0TXD
- removed net N$80: R18.2, U1.CC2
- removed net ROW0: D2.C, D3.C, D4.C, D5.C, U3.GPIO45
- removed net ROW1: D6.C, D7.C, D8.C, D9.C, U3.MTDO
- removed net ROW2: D10.C, D11.C, D12.C, D13.C, U3.GPIO37
- removed net ROW3: D14.C, D15.C, D16.C, D17.C, U3.GPIO36
- removed net ROW4: D18.C, D19.C, D20.C, D21.C, U3.GPIO35
- removed net SD_CLK: SD1.CLK(SCLK), U3.GPIO8
- removed net SD_CMD: SD1.CMD(DI), U3.GPIO9
- removed net SD_D0: SD1.DAT0(DO), U3.GPIO7
- new net MISO: SD1.DAT0(DO), U3.GPIO8
- new net N$37: SW22G$2.1, U3.GPIO0
- new net SW_R1C1: SWR1C1.1, U3.MTMS
- new net SW_R1C2: JP3.1, R18.1, SWR1C2.1
- new net SW_R1C3: SWR1C3.1, U3.U0RXD
- new net SW_R1C4: SWR1C4.1, U3.GPIO45
- new net SW_R2C1: SWR2C1.1, U3.GPIO38
- new net SW_R2C2: SWR2C2.1, U3.MTCK
- new net SW_R2C3: SWR2C3.1, U3.MTDO
- new net SW_R2C4: SWR2C4.1, U3.MTDI
- new net SW_R3C1: SWR3C1.1, U3.GPIO37
- new net SW_R3C2: SWR3C2.1, U3.GPIO36
- new net SW_R3C3: SWR3C3.1, U3.GPIO35
- new net SW_R3C4: SWR3C4.1, U3.GPIO34
- new net SW_R4C1: SWR4C1.1, U3.GPIO21
- new net SW_R4C2: SWR4C2.1, U3.SPICLK_N
- new net SW_R4C3: SWR4C3.1, U3.SPICLK_P
- new net SW_R4C4: SWR4C4.1, U3.GPIO33
- new net SW_R5C1: SWR5C1.1, U3.XTAL_32K_P
- new net SW_R5C2: SWR5C2.1, U3.XTAL_32K_N
- new net SW_R5C3: SWR5C3.1, U3.GPIO17
- new net SW_R5C4: SWR5C4.1, U3.GPIO18
- net +3V3: now also C30.2, U$3.1, U$3.2; no longer U$3.3
- net 12V: now also C32.2
- net CARD_DET: now also U3.GPIO7; no longer U3.GPIO6
- net DC: now also JP5.3, U3.GPIO11; no longer U3.GPIO12
- net GND: now also C30.1, C32.1, JP5.6, R3.2, R4.2, SWR1C1.2, SWR1C2.2, SWR1C3.2, SWR1C4.2, SWR2C1.2, SWR2C2.2, SWR2C3.2, SWR2C4.2, SWR3C1.2, SWR3C2.2, SWR3C3.2, SWR3C4.2, SWR4C1.2, SWR4C2.2, SWR4C3.2, SWR4C4.2, SWR5C1.2, SWR5C2.2, SWR5C3.2, SWR5C4.2; no longer SW4.1, SW4.4, U$3.11, U$3.12, U$3.2, X2.GND@0, X2.GND@1
- net MOSI: now also JP5.5, SD1.CMD(DI)
- net N$1: now also U1.VBUS; no longer JP1.1
- net N$27: now also JP1.1, U3.SPICS1; no longer D5.A, SWR1C4.1
- net N$28: now also R3.1, U1.CC2; no longer SW22G$2.1, SW4.2, SW4.3, U3.GPIO0
- net N$30: now also R4.1, U1.CC1; no longer SW1.S, SW1.S1, U3.GPIO17
- net N$32: now also C29.2, IC2.VIN, JP2.2; no longer R4.2, U1.CC1
- net N$41: no longer R19.1
- net N$44: now also R18.2, U3.U0TXD; no longer D4.A, SWR1C3.1
- net N$46: now also SW1.S, SW1.S1, U3.GPIO13; no longer D2.A, SWR1C1.1
- net N$47: now also SW2.S, SW2.S1, U3.GPIO14; no longer D9.A, SWR2C4.1
- net OLED_CS: now also JP5.1, U3.GPIO12; no longer U3.GPIO14
- net OLED_RESET: now also JP5.2, U3.GPIO6; no longer U3.GPIO13
- net RESET: no longer R19.2
- net SCLK: now also JP5.4, SD1.CLK(SCLK), U3.GPIO9; no longer U3.GPIO11
- net USB_DN: now also U1.DN1, U1.DN2
- net USB_DP: now also U1.DP1, U1.DP2
Other:
- note added: "D0 = SCL = SCLK D1 = SDA = MOSI"
- moved on the sheet: JP3, R12, R17, R18, R3, R4, SW1, SW2, SW22, SWR1C2, SWR1C3, SWR1C4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
