File: pcb/rev2/duckypad.brd (EAGLE design)
At the start: 110 x 96 mm, 158 parts, among them IC2 REG1117, SW1 SPST_TACT-EVQQ2, SW2 SPST_TACT-EVQQ2, SW21 EC12E_SW, SW22 EC12E_SW, SW3 324_SW324_SWITCH_FOOT_HOLE, SW4 324_SW324_SWITCH_FOOT_HOLE, U1 USBC_16P, U2 USBC_16P, U3 ESP32-S3FN8, Y1 16MHz_12pF

Commit message: switching to matrix
Parts:
- removed D10, D11, D12, D13, D14, D15, D16, D17, D18, D19, D2, D20, D21, D22, D23, D3, D4, D5, D6, D7, D8, D9: (no value), adafruit_changed:SOD-123
- removed SW4: 324_SW324_SWITCH_FOOT_HOLE, 3pos_slide_switch:342_SWICH_FOOT_HOLE
- added JP1: (no value), adafruit_changed:1X01-CLEANBIG
- added JP5: (no value), pinhead:2X03
- added R18: 470, joyAnalog:0805
- added U$3: PINHD1X2, adafruit_changed:1X02
- moved SW3 3.49 mm to (108.4, 75.5)
Connections:
- removed net COL0: SWR1C1.1, SWR2C1.1, SWR3C1.1, SWR4C1.1, SWR5C1.1
- removed net COL1: SWR1C2.1, SWR2C2.1, SWR3C2.1, SWR4C2.1, SWR5C2.1
- removed net COL2: SWR1C3.1, SWR2C3.1, SWR3C3.1, SWR4C3.1, SWR5C3.1
- removed net COL3: SWR1C4.1, SWR2C4.1, SWR3C4.1, SWR4C4.1, SWR5C4.1
- removed net COL4: SW1.A, SW1.A', SW2.A, SW2.A'
- removed net N$45: D3.A, SWR1C2.2
- removed net N$50: D8.A, SWR2C3.2
- removed net N$51: D7.A, SWR2C2.2
- removed net N$52: D6.A, SWR2C1.2
- removed net N$53: D10.A, SWR3C4.2
- removed net N$54: D11.A, SWR3C3.2
- removed net N$55: D12.A, SWR3C2.2
- removed net N$56: D13.A, SWR3C1.2
- removed net N$57: D17.A, SWR4C4.2
- removed net N$58: D16.A, SWR4C3.2
- removed net N$59: D15.A, SWR4C2.2
- removed net N$60: D14.A, SWR4C1.2
- removed net N$61: D18.A, SWR5C4.2
- removed net N$62: D19.A, SWR5C3.2
- removed net N$63: D20.A, SWR5C2.2
- removed net N$64: D21.A, SWR5C1.2
- removed net N$65: D22.A, SW1.B, SW1.B'
- removed net N$66: D23.A, SW2.B, SW2.B'
- removed net ROW0: D2.C, D3.C, D4.C, D5.C
- removed net ROW1: D6.C, D7.C, D8.C, D9.C
- removed net ROW2: D10.C, D11.C, D12.C, D13.C
- removed net ROW3: D14.C, D15.C, D16.C, D17.C, D22.C
- removed net ROW4: D18.C, D19.C, D20.C, D21.C, D23.C
- new net SW_R1C1: SWR1C1.2, U3.48
- new net SW_R1C2: JP3.1, R18.1, SWR1C2.2
- new net SW_R1C3: SWR1C3.2, U3.50
- new net SW_R1C4: SWR1C4.2, U3.51
- new net SW_R2C1: SWR2C1.2, U3.43
- new net SW_R2C2: SWR2C2.2, U3.44
- new net SW_R2C3: SWR2C3.2, U3.45
- new net SW_R2C4: SWR2C4.2, U3.47
- new net SW_R3C1: SWR3C1.2, U3.42
- new net SW_R3C2: SWR3C2.2, U3.41
- new net SW_R3C3: SWR3C3.2, U3.40
- new net SW_R3C4: SWR3C4.2, U3.39
- new net SW_R4C1: SWR4C1.2, U3.27
- new net SW_R4C2: SWR4C2.2, U3.36
- new net SW_R4C3: SWR4C3.2, U3.37
- new net SW_R4C4: SWR4C4.2, U3.38
- new net SW_R5C1: SWR5C1.2, U3.21
- new net SW_R5C2: SWR5C2.2, U3.22
- new net SW_R5C3: SWR5C3.2, U3.23
- new net SW_R5C4: SWR5C4.2, U3.24
- net +3V3: now also U$3.1, U$3.2
- net DC: now also JP5.3
- net GND: now also JP5.6, SW1.A, SW1.A', SW2.A, SW2.A', SWR1C1.1, SWR1C2.1, SWR1C3.1, SWR1C4.1, SWR2C1.1, SWR2C2.1, SWR2C3.1, SWR2C4.1, SWR3C1.1, SWR3C2.1, SWR3C3.1, SWR3C4.1, SWR4C1.1, SWR4C2.1, SWR4C3.1, SWR4C4.1, SWR5C1.1, SWR5C2.1, SWR5C3.1, SWR5C4.1
- net MOSI: now also JP5.5
- net N$27: now also JP1.1, U3.28; no longer D5.A, SWR1C4.2
- net N$29: now also U3.52
- net N$44: now also R18.2, U3.49; no longer D4.A, SWR1C3.2
- net N$46: now also SW1.B, SW1.B', U3.18; no longer D2.A, SWR1C1.2
- net N$47: now also SW2.B, SW2.B', U3.19; no longer D9.A, SWR2C4.2
- net OLED_CS: now also JP5.1
- net OLED_RESET: now also JP5.2
- net SCLK: now also JP5.4
Routing:
- net SW_R5C1: track 0.00 -> 111.2 mm
- net SW_R4C1: track 0.00 -> 97.8 mm
- net SW_R1C1: track 0.00 -> 93.2 mm
- net SW_R5C2: track 0.00 -> 91.3 mm
- net SW_R4C2: track 0.00 -> 78.7 mm
- net SW_R2C1: track 0.00 -> 75.8 mm
- net SW_R5C3: track 0.00 -> 71.0 mm
- net N$44: track 0.00 -> 65.5 mm
- net SW_R3C1: track 0.00 -> 64.2 mm
- net N$46: track 0.00 -> 58.8 mm, vias 0 -> 1
- net SW_R4C3: track 0.00 -> 56.2 mm
- net SW_R2C2: track 0.00 -> 55.1 mm
- net N$47: track 0.00 -> 48.4 mm, vias 0 -> 1
- net SW_R3C2: track 0.00 -> 45.2 mm
- net SW_R1C3: track 0.00 -> 45.2 mm
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
Commit message: working on new PCB revision
Parts:
- removed JP1: (no value), adafruit_changed:1X01-CLEANBIG
- removed JP5: (no value), pinhead:2X03
- added D10, D11, D12, D13, D14, D15, D16, D17, D18, D19, D2, D20, D21, D3, D4, D5, D6, D7, D8, D9: 1N4148, duckypad:ADAFRUIT_CHANGED_SOD-123
- added R19: DNP, joyAnalog:0805
- added SW4: 324_SW324_SWITCH_FOOT_HOLE, 3pos_slide_switch:342_SWICH_FOOT_HOLE
- added U5: W25Q32FVSS, SparkFun-DigitalIC:SOIC-8
- added X2: (no value), adafruit_changed:U.FL
- C1, C10, C2, C9: value 10nF -> 100nF
- C27: value 47uF -> 100uF
- C29: value 10uF -> 4.7uF
- C30: value 100nF -> 1uF
- C31: value 4.7uF -> 100nF
- C34, C38: value 2.2uF -> 4.7uF
- C35: value 22pF -> 12pF
- C4: value 1uF -> 100nF
- C46: value 100nF -> 4.7uF
- D1: value (none) -> 1N4148; device adafruit_changed:SOD-123 -> duckypad:ADAFRUIT_CHANGED_SOD-123
- L2: value PRS4018-4R7MT -> 4.7uH
- R13, R14, R15, R8: value 10K -> 5K1
- R2: value 10K -> 62K
- R3: value 5.1K -> (none); device joyAnalog:0805 -> adafruit_changed:R2010
- R4: value 5.1K -> 470
- R5: value 5.1K -> 10K
- R6, R7: value 560K -> 510K
- U$3: value PINHD1X2 -> SH10P; device adafruit_changed:1X02 -> duckypad:DUCKYPAD_SM12B-SSR-H-TB
- moved JP3 114.5 mm to (107.4, 2.16)
- moved R18 87.1 mm to (100.3, 20.1), turned to 90 degrees
- moved U$3 65.0 mm to (108.0, 11.7), flipped to the bottom, turned to 270 degrees
- moved C33 58.6 mm to (83.3, 16.2), flipped to the bottom, turned to 90 degrees
- moved U$19 55.6 mm to (86.9, 16.2), flipped to the bottom, turned to 270 degrees
- moved L2 54.1 mm to (85.0, 20.1), flipped to the bottom, turned to 180 degrees
- moved R10 52.8 mm to (90.0, 16.2), flipped to the bottom, turned to 90 degrees
- moved C35 51.5 mm to (92.1, 16.2), flipped to the bottom, turned to 90 degrees
- moved D1 50.5 mm to (90.2, 19.1), flipped to the bottom, turned to 0 degrees
- moved R7 50.3 mm to (94.1, 16.2), flipped to the bottom, turned to 270 degrees
- moved C46 46.9 mm to (94.9, 18.9), flipped to the bottom, turned to 0 degrees
- moved C31 45.5 mm to (95.9, 21.5), flipped to the bottom, turned to 0 degrees
- moved C32 35.2 mm to (74.2, 57.9), flipped to the top, turned to 270 degrees
- moved R5 17.6 mm to (69.7, 94.2), turned to 180 degrees
- moved R3 17.3 mm to (92.7, 1.52)
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Connections:
- removed net MISO: SD1.7, U3.13
- removed net N$37: SW22.D, U3.5
- removed net SW_R1C1: SWR1C1.2, U3.48
- removed net SW_R1C2: JP3.1, R18.1, SWR1C2.2
- removed net SW_R1C3: SWR1C3.2, U3.50
- removed net SW_R1C4: SWR1C4.2, U3.51
- removed net SW_R2C1: SWR2C1.2, U3.43
- removed net SW_R2C2: SWR2C2.2, U3.44
- removed net SW_R2C3: SWR2C3.2, U3.45
- removed net SW_R2C4: SWR2C4.2, U3.47
- removed net SW_R3C1: SWR3C1.2, U3.42
- removed net SW_R3C2: SWR3C2.2, U3.41
- removed net SW_R3C3: SWR3C3.2, U3.40
- removed net SW_R3C4: SWR3C4.2, U3.39
- removed net SW_R4C1: SWR4C1.2, U3.27
- removed net SW_R4C2: SWR4C2.2, U3.36
- removed net SW_R4C3: SWR4C3.2, U3.37
- removed net SW_R4C4: SWR4C4.2, U3.38
- removed net SW_R5C1: SWR5C1.2, U3.21
- removed net SW_R5C2: SWR5C2.2, U3.22
- removed net SW_R5C3: SWR5C3.2, U3.23
- removed net SW_R5C4: SWR5C4.2, U3.24
- new net AUX_DN: U1.A7, U1.B7, U3.21
- new net AUX_DP: U1.A6, U1.B6, U3.22
- new net CC_BUSY: R18.1, R4.1, U$3.4, U3.27
- new net COL0: SWR1C1.1, SWR2C1.1, SWR3C1.1, SWR4C1.1, SWR5C1.1, U3.48
- new net COL1: SWR1C2.1, SWR2C2.1, SWR3C2.1, SWR4C2.1, SWR5C2.1, U3.47
- new net COL2: SWR1C3.1, SWR2C3.1, SWR3C3.1, SWR4C3.1, SWR5C3.1, U3.44
- new net COL3: SWR1C4.1, SWR2C4.1, SWR3C4.1, SWR4C4.1, SWR5C4.1, U3.43
- new net N$45: D3.A, SWR1C2.2
- new net N$50: D8.A, SWR2C3.2
- new net N$51: D7.A, SWR2C2.2
- new net N$52: D6.A, SWR2C1.2
- new net N$53: D10.A, SWR3C4.2
- new net N$54: D11.A, SWR3C3.2
- new net N$55: D12.A, SWR3C2.2
- new net N$56: D13.A, SWR3C1.2
- new net N$57: D17.A, SWR4C4.2
- new net N$58: D16.A, SWR4C3.2
- new net N$59: D15.A, SWR4C2.2
- new net N$60: D14.A, SWR4C1.2
- new net N$61: D18.A, SWR5C4.2
- new net N$62: D19.A, SWR5C3.2
- new net N$63: D20.A, SWR5C2.2
- new net N$64: D21.A, SWR5C1.2
- new net N$65: SW2.B, SW2.B', U3.24
- new net N$66: C29.2, IC2.3, JP2.2, U$3.1, U1.A4B9, U1.B4A9
- new net N$67: U$3.5, U3.36
- new net N$68: U$3.6, U3.37
- new net N$69: U$3.7, U3.38
- new net N$70: U$3.8, U3.39
- new net N$71: R3.1, X2.3
- new net N$72: U$3.9, U3.50
- new net N$73: JP3.1, U$3.10, U3.49
- new net N$74: U3.33, U5.6
- new net N$75: U3.30, U5.7
- new net N$76: U3.31, U5.3
- new net N$77: U3.32, U5.1
- new net N$78: U3.34, U5.2
- new net N$79: U3.35, U5.5
- new net N$80: R18.2, U1.B5
- new net ROW0: D2.C, D3.C, D4.C, D5.C, U3.51
- new net ROW1: D6.C, D7.C, D8.C, D9.C, U3.45
- new net ROW2: D10.C, D11.C, D12.C, D13.C, U3.42
- new net ROW3: D14.C, D15.C, D16.C, D17.C, U3.41
- new net ROW4: D18.C, D19.C, D20.C, D21.C, U3.40
- new net SD_CLK: SD1.5, U3.13
- new net SD_CMD: SD1.3, U3.14
- new net SD_D0: SD1.7, U3.12
- net +3V3: now also C32.2, U$3.3, U5.8; no longer U$3.1, U$3.2
- net 12V: no longer C32.2
- net CARD_DET: now also U3.11; no longer U3.12
- net DC: now also U3.17; no longer JP5.3, U3.16
- net GND: now also SW4.P$1, SW4.P$4, U$3.2, U$3.FIT@1, U$3.FIT@2, U5.4, X2.1, X2.2; no longer JP5.6, R3.2, R4.2, SWR1C1.1, SWR1C2.1, SWR1C3.1, SWR1C4.1, SWR2C1.1, SWR2C2.1, SWR2C3.1, SWR2C4.1, SWR3C1.1, SWR3C2.1, SWR3C3.1, SWR3C4.1, SWR4C1.1, SWR4C2.1, SWR4C3.1, SWR4C4.1, SWR5C1.1, SWR5C2.1, SWR5C3.1, SWR5C4.1
- net MOSI: no longer JP5.5, SD1.3
- net N$1: no longer U1.A4B9, U1.B4A9
- net N$27: now also D5.A, SWR1C4.2; no longer JP1.1, U3.28
- net N$28: now also SW22.D, SW4.P$2, SW4.P$3, U3.5; no longer R3.1, U1.B5
- net N$30: now also SW1.B, SW1.B', U3.23; no longer R4.1, U1.A5
- net N$32: now also R4.2, U1.A5; no longer C29.2, IC2.3, JP2.2
- net N$41: now also R19.1
- net N$44: now also D4.A, SWR1C3.2; no longer R18.2, U3.49
- net N$46: now also D2.A, SWR1C1.2; no longer SW1.B, SW1.B', U3.18
- net N$47: now also D9.A, SWR2C4.2; no longer SW2.B, SW2.B', U3.19
- net OLED_CS: now also U3.19; no longer JP5.1, U3.17
- net OLED_RESET: now also U3.18; no longer JP5.2, U3.11
- net RESET: now also R19.2
- net SCLK: now also U3.16; no longer JP5.4, SD1.5, U3.14
- net USB_DN: no longer U1.A7, U1.B7
- net USB_DP: no longer U1.A6, U1.B6
Routing:
- net +3V3: track 619.7 -> 191.7 mm, vias 25 -> 33
- net N$1: track 330.9 -> 17.3 mm, vias 2 -> 0
- net USB_DP: track 340.6 -> 51.4 mm, vias 1 -> 2
- net USB_DN: track 323.0 -> 54.0 mm, vias 1 -> 2
- net COL0: track 0.00 -> 205.9 mm, vias 0 -> 6
- net COL1: track 0.00 -> 180.2 mm, vias 0 -> 6
- net COL2: track 0.00 -> 148.5 mm, vias 0 -> 6
- net N$66: track 0.00 -> 117.3 mm, vias 0 -> 1
- net N$73: track 0.00 -> 115.1 mm, vias 0 -> 1
- net ROW3: track 0.00 -> 111.4 mm
- net SW_R5C1: track 111.2 -> 0.00 mm
- net N$72: track 0.00 -> 109.4 mm, vias 0 -> 2
- net ROW4: track 0.00 -> 108.8 mm
- net COL3: track 0.00 -> 104.8 mm, vias 0 -> 5
- net SW_R4C1: track 97.8 -> 0.00 mm
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- added copper zone on layer 2, net +3V3
- added copper zone on layer 15, net GND
- added copper zone on layer 15, net WTF2
- added copper zone on layer 2, net WTF2
Other:
- board text added: "duckyPad Pro PT3 dekuNukem JUN2024"
- board text added: "watch out for strapping pins GPIO3 must have pull resistor, pull to high to free up JTAG pins? 3.5mm corner radius double check RESET jumper has NO PASTE"
- board text removed: "CS"
- board text removed: "DC"
- board text removed: "GND"
- board text removed: "MOSI"
- board text removed: "RST"
- board text removed: "SCK"
- board text removed: "SPICS1"
- board text removed: "duckyPad Pro PT2 dekuNukem MAY2024"
- board text removed: "watch out for strapping pins GPIO3 must have pull resistor, pull to high to free up JTAG pins? 3.5mm corner radius MOVED: MOSI SCLK MISO CARD_DET OLED_RESET (new)"
