File: pcb/rev2/duckypad.sch (EAGLE design)
At the start: 158 parts, among them IC2 REG1117, SW1 SPST_TACT-EVQQ2, SW2 SPST_TACT-EVQQ2, SW21 EC12E_SW, SW22 EC12E_SW, SW3 324_SW324_SWITCH_FOOT_HOLE, SW4 324_SW324_SWITCH_FOOT_HOLE, U1 USBC_16P, U2 USBC_16P, U3 ESP32-S3FN8, Y1 16MHz_12pF

Commit message: switching to matrix
Parts:
- removed D10, D11, D12, D13, D14, D15, D16, D17, D18, D19, D2, D20, D21, D22, D23, D3, D4, D5, D6, D7, D8, D9: (no value), adafruit_changed:DIODESOD-123
- removed SW4: 324_SW324_SWITCH_FOOT_HOLE, 3pos_slide_switch:324_SW324_SWITCH_FOOT_HOLE
- added JP1: (no value), adafruit_changed:PINHD-1X1CB
- added JP5: (no value), pinhead:PINHD-2X3
- added R18: 470, joyAnalog:RESISTOR0805-RES
- added U$3: PINHD1X2, adafruit_changed:PINHD1X2
Connections:
- removed net COL0: SWR1C1.2, SWR2C1.2, SWR3C1.2, SWR4C1.2, SWR5C1.2
- removed net COL1: SWR1C2.2, SWR2C2.2, SWR3C2.2, SWR4C2.2, SWR5C2.2
- removed net COL2: SWR1C3.2, SWR2C3.2, SWR3C3.2, SWR4C3.2, SWR5C3.2
- removed net COL3: SWR1C4.2, SWR2C4.2, SWR3C4.2, SWR4C4.2, SWR5C4.2
- removed net COL4: SW1.P, SW1.P1, SW2.P, SW2.P1
- removed net N$45: D3.A, SWR1C2.1
- removed net N$50: D8.A, SWR2C3.1
- removed net N$51: D7.A, SWR2C2.1
- removed net N$52: D6.A, SWR2C1.1
- removed net N$53: D10.A, SWR3C4.1
- removed net N$54: D11.A, SWR3C3.1
- removed net N$55: D12.A, SWR3C2.1
- removed net N$56: D13.A, SWR3C1.1
- removed net N$57: D17.A, SWR4C4.1
- removed net N$58: D16.A, SWR4C3.1
- removed net N$59: D15.A, SWR4C2.1
- removed net N$60: D14.A, SWR4C1.1
- removed net N$61: D18.A, SWR5C4.1
- removed net N$62: D19.A, SWR5C3.1
- removed net N$63: D20.A, SWR5C2.1
- removed net N$64: D21.A, SWR5C1.1
- removed net N$65: D22.A, SW1.S, SW1.S1
- removed net N$66: D23.A, SW2.S, SW2.S1
- removed net ROW0: D2.C, D3.C, D4.C, D5.C
- removed net ROW1: D6.C, D7.C, D8.C, D9.C
- removed net ROW2: D10.C, D11.C, D12.C, D13.C
- removed net ROW3: D14.C, D15.C, D16.C, D17.C, D22.C
- removed net ROW4: D18.C, D19.C, D20.C, D21.C, D23.C
- new net SW_R1C1: SWR1C1.1, U3.MTMS
- new net SW_R1C2: JP3.1, R18.1, SWR1C2.1
- new net SW_R1C3: SWR1C3.1, U3.U0RXD
- new net SW_R1C4: SWR1C4.1, U3.GPIO45
- new net SW_R2C1: SWR2C1.1, U3.GPIO38
- new net SW_R2C2: SWR2C2.1, U3.MTCK
- new net SW_R2C3: SWR2C3.1, U3.MTDO
- new net SW_R2C4: SWR2C4.1, U3.MTDI
- new net SW_R3C1: SWR3C1.1, U3.GPIO37
- new net SW_R3C2: SWR3C2.1, U3.GPIO36
- new net SW_R3C3: SWR3C3.1, U3.GPIO35
- new net SW_R3C4: SWR3C4.1, U3.GPIO34
- new net SW_R4C1: SWR4C1.1, U3.GPIO21
- new net SW_R4C2: SWR4C2.1, U3.SPICLK_N
- new net SW_R4C3: SWR4C3.1, U3.SPICLK_P
- new net SW_R4C4: SWR4C4.1, U3.GPIO33
- new net SW_R5C1: SWR5C1.1, U3.XTAL_32K_P
- new net SW_R5C2: SWR5C2.1, U3.XTAL_32K_N
- new net SW_R5C3: SWR5C3.1, U3.GPIO17
- new net SW_R5C4: SWR5C4.1, U3.GPIO18
- net +3V3: now also U$3.1, U$3.2
- net DC: now also JP5.3
- net GND: now also JP5.6, SW1.P, SW1.P1, SW2.P, SW2.P1, SWR1C1.2, SWR1C2.2, SWR1C3.2, SWR1C4.2, SWR2C1.2, SWR2C2.2, SWR2C3.2, SWR2C4.2, SWR3C1.2, SWR3C2.2, SWR3C3.2, SWR3C4.2, SWR4C1.2, SWR4C2.2, SWR4C3.2, SWR4C4.2, SWR5C1.2, SWR5C2.2, SWR5C3.2, SWR5C4.2
- net MOSI: now also JP5.5
- net N$27: now also JP1.1, U3.SPICS1; no longer D5.A, SWR1C4.1
- net N$29: now also U3.GPIO46
- net N$44: now also R18.2, U3.U0TXD; no longer D4.A, SWR1C3.1
- net N$46: now also SW1.S, SW1.S1, U3.GPIO13; no longer D2.A, SWR1C1.1
- net N$47: now also SW2.S, SW2.S1, U3.GPIO14; no longer D9.A, SWR2C4.1
- net OLED_CS: now also JP5.1
- net OLED_RESET: now also JP5.2
- net SCLK: now also JP5.4
Other:
- moved on the sheet: SW1, SW2, SWR1C2, SWR1C3, SWR1C4, SWR2C2, SWR2C3, SWR2C4, SWR3C2, SWR3C3, SWR3C4, SWR4C2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

Commit message: working on new PCB revision
Parts:
- removed JP1: (no value), adafruit_changed:PINHD-1X1CB
- removed JP5: (no value), pinhead:PINHD-2X3
- added D10, D11, D12, D13, D14, D15, D16, D17, D18, D19, D2, D20, D21, D3, D4, D5, D6, D7, D8, D9: 1N4148, duckypad:ADAFRUIT_CHANGED_DIODESOD-123
- added R19: DNP, joyAnalog:RESISTOR0805-RES
- added SW4: 324_SW324_SWITCH_FOOT_HOLE, 3pos_slide_switch:324_SW324_SWITCH_FOOT_HOLE
- added U5: W25Q32FVSS, SparkFun-DigitalIC:W25Q32FVSS
- added X2: (no value), adafruit_changed:ANTENNA_U.FL
- C1, C10, C2, C9: value 10nF -> 100nF
- C27: value 47uF -> 100uF
- C29: value 10uF -> 4.7uF
- C30: value 100nF -> 1uF
- C31: value 4.7uF -> 100nF
- C34, C38: value 2.2uF -> 4.7uF
- C35: value 22pF -> 12pF
- C4: value 1uF -> 100nF
- C46: value 100nF -> 4.7uF
- D1: value (none) -> 1N4148; device adafruit_changed:DIODESOD-123 -> duckypad:ADAFRUIT_CHANGED_DIODESOD-123
- L2: value PRS4018-4R7MT -> 4.7uH
- R13, R14, R15, R8: value 10K -> 5K1
- R2: value 10K -> 62K
- R3: value 5.1K -> (none); device joyAnalog:RESISTOR0805-RES -> adafruit_changed:R-US_R2010
- R4: value 5.1K -> 470
- R5: value 5.1K -> 10K
- R6, R7: value 560K -> 510K
- U$3: value PINHD1X2 -> SH10P; device adafruit_changed:PINHD1X2 -> duckypad:SH10P
Connections:
- removed net MISO: SD1.DAT0(DO), U3.GPIO8
- removed net N$37: SW22G$2.1, U3.GPIO0
- removed net SW_R1C1: SWR1C1.1, U3.MTMS
- removed net SW_R1C2: JP3.1, R18.1, SWR1C2.1
- removed net SW_R1C3: SWR1C3.1, U3.U0RXD
- removed net SW_R1C4: SWR1C4.1, U3.GPIO45
- removed net SW_R2C1: SWR2C1.1, U3.GPIO38
- removed net SW_R2C2: SWR2C2.1, U3.MTCK
- removed net SW_R2C3: SWR2C3.1, U3.MTDO
- removed net SW_R2C4: SWR2C4.1, U3.MTDI
- removed net SW_R3C1: SWR3C1.1, U3.GPIO37
- removed net SW_R3C2: SWR3C2.1, U3.GPIO36
- removed net SW_R3C3: SWR3C3.1, U3.GPIO35
- removed net SW_R3C4: SWR3C4.1, U3.GPIO34
- removed net SW_R4C1: SWR4C1.1, U3.GPIO21
- removed net SW_R4C2: SWR4C2.1, U3.SPICLK_N
- removed net SW_R4C3: SWR4C3.1, U3.SPICLK_P
- removed net SW_R4C4: SWR4C4.1, U3.GPIO33
- removed net SW_R5C1: SWR5C1.1, U3.XTAL_32K_P
- removed net SW_R5C2: SWR5C2.1, U3.XTAL_32K_N
- removed net SW_R5C3: SWR5C3.1, U3.GPIO17
- removed net SW_R5C4: SWR5C4.1, U3.GPIO18
- new net AUX_DN: U1.DN1, U1.DN2, U3.XTAL_32K_P
- new net AUX_DP: U1.DP1, U1.DP2, U3.XTAL_32K_N
- new net CC_BUSY: R18.1, R4.1, U$3.4, U3.GPIO21
- new net COL0: SWR1C1.2, SWR2C1.2, SWR3C1.2, SWR4C1.2, SWR5C1.2, U3.MTMS
- new net COL1: SWR1C2.2, SWR2C2.2, SWR3C2.2, SWR4C2.2, SWR5C2.2, U3.MTDI
- new net COL2: SWR1C3.2, SWR2C3.2, SWR3C3.2, SWR4C3.2, SWR5C3.2, U3.MTCK
- new net COL3: SWR1C4.2, SWR2C4.2, SWR3C4.2, SWR4C4.2, SWR5C4.2, U3.GPIO38
- new net N$45: D3.A, SWR1C2.1
- new net N$50: D8.A, SWR2C3.1
- new net N$51: D7.A, SWR2C2.1
- new net N$52: D6.A, SWR2C1.1
- new net N$53: D10.A, SWR3C4.1
- new net N$54: D11.A, SWR3C3.1
- new net N$55: D12.A, SWR3C2.1
- new net N$56: D13.A, SWR3C1.1
- new net N$57: D17.A, SWR4C4.1
- new net N$58: D16.A, SWR4C3.1
- new net N$59: D15.A, SWR4C2.1
- new net N$60: D14.A, SWR4C1.1
- new net N$61: D18.A, SWR5C4.1
- new net N$62: D19.A, SWR5C3.1
- new net N$63: D20.A, SWR5C2.1
- new net N$64: D21.A, SWR5C1.1
- new net N$65: SW2.S, SW2.S1, U3.GPIO18
- new net N$66: C29.2, IC2.VIN, JP2.2, U$3.1, U1.VBUS
- new net N$67: U$3.5, U3.SPICLK_N
- new net N$68: U$3.6, U3.SPICLK_P
- new net N$69: U$3.7, U3.GPIO33
- new net N$70: U$3.8, U3.GPIO34
- new net N$71: R3.1, X2.SIGNAL
- new net N$72: U$3.9, U3.U0RXD
- new net N$73: JP3.1, U$3.10, U3.U0TXD
- new net N$74: U3.SPICLK, U5.SCK
- new net N$75: U3.SPIHD, U5.!HOLD!(D3)
- new net N$76: U3.SPIWP, U5.!WP!(D2)
- new net N$77: U3.SPICS0, U5.!CS!
- new net N$78: U3.SPIQ, U5.SO(D1)
- new net N$79: U3.SPID, U5.SI(D0)
- new net N$80: R18.2, U1.CC2
- new net ROW0: D2.C, D3.C, D4.C, D5.C, U3.GPIO45
- new net ROW1: D6.C, D7.C, D8.C, D9.C, U3.MTDO
- new net ROW2: D10.C, D11.C, D12.C, D13.C, U3.GPIO37
- new net ROW3: D14.C, D15.C, D16.C, D17.C, U3.GPIO36
- new net ROW4: D18.C, D19.C, D20.C, D21.C, U3.GPIO35
- new net SD_CLK: SD1.CLK(SCLK), U3.GPIO8
- new net SD_CMD: SD1.CMD(DI), U3.GPIO9
- new net SD_D0: SD1.DAT0(DO), U3.GPIO7
- net +3V3: now also C32.2, U$3.3, U5.VCC; no longer U$3.1, U$3.2
- net 12V: no longer C32.2
- net CARD_DET: now also U3.GPIO6; no longer U3.GPIO7
- net DC: now also U3.GPIO12; no longer JP5.3, U3.GPIO11
- net GND: now also SW4.1, SW4.4, U$3.11, U$3.12, U$3.2, U5.GND, X2.GND@0, X2.GND@1; no longer JP5.6, R3.2, R4.2, SWR1C1.2, SWR1C2.2, SWR1C3.2, SWR1C4.2, SWR2C1.2, SWR2C2.2, SWR2C3.2, SWR2C4.2, SWR3C1.2, SWR3C2.2, SWR3C3.2, SWR3C4.2, SWR4C1.2, SWR4C2.2, SWR4C3.2, SWR4C4.2, SWR5C1.2, SWR5C2.2, SWR5C3.2, SWR5C4.2
- net MOSI: no longer JP5.5, SD1.CMD(DI)
- net N$1: no longer U1.VBUS
- net N$27: now also D5.A, SWR1C4.1; no longer JP1.1, U3.SPICS1
- net N$28: now also SW22G$2.1, SW4.2, SW4.3, U3.GPIO0; no longer R3.1, U1.CC2
- net N$30: now also SW1.S, SW1.S1, U3.GPIO17; no longer R4.1, U1.CC1
- net N$32: now also R4.2, U1.CC1; no longer C29.2, IC2.VIN, JP2.2
- net N$41: now also R19.1
- net N$44: now also D4.A, SWR1C3.1; no longer R18.2, U3.U0TXD
- net N$46: now also D2.A, SWR1C1.1; no longer SW1.S, SW1.S1, U3.GPIO13
- net N$47: now also D9.A, SWR2C4.1; no longer SW2.S, SW2.S1, U3.GPIO14
- net OLED_CS: now also U3.GPIO14; no longer JP5.1, U3.GPIO12
- net OLED_RESET: now also U3.GPIO13; no longer JP5.2, U3.GPIO6
- net RESET: now also R19.2
- net SCLK: now also U3.GPIO11; no longer JP5.4, SD1.CLK(SCLK), U3.GPIO9
- net USB_DN: no longer U1.DN1, U1.DN2
- net USB_DP: no longer U1.DP1, U1.DP2
Other:
- note removed: "D0 = SCL = SCLK D1 = SDA = MOSI"
- moved on the sheet: C30, C32, JP3, R12, R17, R18, R3, R4, SW1, SW2, SW22, SWR1C2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
