File: pcb/plate/bottom.brd (EAGLE design)
At the start: 110 x 96 mm, 8 parts

Commit message: update plates
Parts:
- moved U$10 1.00 mm to (91.8, 7.00)
- moved U$12 1.00 mm to (38.5, 38.5)
- moved U$13 1.00 mm to (57.5, 19.5)
- moved U$17 1.00 mm to (99.0, 76.5)
- moved U$8 1.00 mm to (38.5, 57.5)
- moved U$9 1.00 mm to (57.5, 76.5)
- moved U$14 0.50 mm to (19.0, 76.5)
- moved U$22 0.50 mm to (19.0, 19.5)
Other:
- board size 110 x 96 mm -> 109 x 96 mm
Changed lines of the file:
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@@
 <grid distance="5" unitdist="mil" unit="mil" style="lines" multiple="1" display="yes" altdistance="1" altunitdist="mil" altunit="mil"/>
 <layers>
-<layer number="1" name="Top" color="4" fill="1" visible="no" active="yes"/>
+<layer number="1" name="Top" color="4" fill="1" visible="yes" active="yes"/>
 <layer number="2" name="pwr" color="49" fill="1" visible="no" active="yes"/>
 <layer number="3" name="Route3" color="4" fill="3" visible="no" active="no"/>
@@
 <layer number="19" name="Unrouted" color="6" fill="1" visible="yes" active="yes"/>
 <layer number="20" name="Dimension" color="15" fill="1" visible="yes" active="yes"/>
-<layer number="21" name="tPlace" color="7" fill="1" visible="no" active="yes"/>
+<layer number="21" name="tPlace" color="7" fill="1" visible="yes" active="yes"/>
 <layer number="22" name="bPlace" color="7" fill="1" visible="yes" active="yes"/>
-<layer number="23" name="tOrigins" color="15" fill="1" visible="no" active="yes"/>
+<layer number="23" name="tOrigins" color="15" fill="1" visible="yes" active="yes"/>
 <layer number="24" name="bOrigins" color="15" fill="1" visible="yes" active="yes"/>
-<layer number="25" name="tNames" color="7" fill="1" visible="no" active="yes"/>
+<layer number="25" name="tNames" color="7" fill="1" visible="yes" active="yes"/>
 <layer number="26" name="bNames" color="7" fill="1" visible="yes" active="yes"/>
-<layer number="27" name="tValues" color="7" fill="1" visible="no" active="yes"/>
-<layer number="28" name="bValues" color="7" fill="1" visible="no" active="yes"/>
+<layer number="27" name="tValues" color="7" fill="1" visible="yes" active="yes"/>
+<layer number="28" name="bValues" color="7" fill="1" visible="yes" active="yes"/>
 <layer number="29" name="tStop" color="7" fill="3" visible="no" active="yes"/>
 <layer number="30" name="bStop" color="7" fill="6" visible="no" active="yes"/>
@@
 <layer number="37" name="tTest" color="7" fill="1" visible="no" active="yes"/>
 <layer number="38" name="bTest" color="7" fill="1" visible="no" active="yes"/>
-<layer number="39" name="tKeepout" color="4" fill="11" visible="no" active="yes"/>
+<layer number="39" name="tKeepout" color="4" fill="11" visible="yes" active="yes"/>
 <layer number="40" name="bKeepout" color="1" fill="11" visible="yes" active="yes"/>
-<layer number="41" name="tRestrict" color="4" fill="10" visible="no" active="yes"/>
+<layer number="41" name="tRestrict" color="4" fill="10" visible="yes" active="yes"/>
 <layer number="42" name="bRestrict" color="1" fill="10" visible="yes" active="yes"/>
 <layer number="43" name="vRestrict" color="2" fill="10" visible="no" active="yes"/>
@@
 <layer number="49" name="Reference" color="7" fill="1" visible="no" active="yes"/>
 <layer number="50" name="dxf" color="7" fill="1" visible="no" active="no"/>
-<layer number="51" name="tDocu" color="7" fill="1" visible="no" active="yes"/>
+<layer number="51" name="tDocu" color="7" fill="1" visible="yes" active="yes"/>
 <layer number="52" name="bDocu" color="7" fill="1" visible="yes" active="yes"/>
 <layer number="53" name="tGND_GNDA" color="7" fill="9" visible="no" active="no"/>
@@
 <board>
 <plain>
-<wire x1="3.5" y1="0" x2="106.5" y2="0" width="0" layer="20"/>
-<wire x1="106.5" y1="0" x2="110" y2="3.5" width="0" layer="20" curve="90"/>
-<wire x1="110" y1="3.5" x2="110" y2="92.5" width="0" layer="20"/>
-<wire x1="110" y1="92.5" x2="106.5" y2="96" width="0" layer="20" curve="90"/>
-<wire x1="106.5" y1="96" x2="3.5" y2="96" width="0" layer="20"/>
-<wire x1="3.5" y1="96" x2="0" y2="92.5" width="0" layer="20" curve="90"/>
-<wire x1="0" y1="92.5" x2="0" y2="3.5" width="0" layer="20"/>
+<wire x1="0" y1="3.5" x2="0" y2="92.5" width="0" layer="20"/>
+<wire x1="0" y1="92.5" x2="3.5" y2="96" width="0" layer="20" curve="-90"/>
+<wire x1="3.5" y1="96" x2="70.5" y2="96" width="0" layer="20"/>
+<wire x1="70.5" y1="96" x2="72" y2="94.5" width="0" layer="20" curve="-90"/>
+<wire x1="72" y1="94.5" x2="72" y2="93.5" width="0" layer="20"/>
+<wire x1="72" y1="93.5" x2="73.5" y2="92" width="0" layer="20" curve="90"/>
+<wire x1="73.5" y1="92" x2="81.5" y2="92" width="0" layer="20"/>
+<wire x1="81.5" y1="92" x2="83" y2="93.5" width="0" layer="20" curve="90"/>
+<wire x1="83" y1="93.5" x2="83" y2="94.5" width="0" layer="20"/>
+<wire x1="83" y1="94.5" x2="84.5" y2="96" width="0" layer="20" curve="-90"/>
+<wire x1="84.5" y1="96" x2="105.5" y2="96" width="0" layer="20"/>
 <wire x1="0" y1="3.5" x2="3.5" y2="0" width="0" layer="20" curve="90"/>
+<wire x1="104" y1="16.5" x2="104" y2="6.5" width="0" layer="20"/>
+<wire x1="104" y1="6.5" x2="105.5" y2="5.127" width="0" layer="20" curve="90"/>
+<wire x1="105.5" y1="5.127" x2="107.5" y2="5.127" width="0" layer="20"/>
+<wire x1="107.5" y1="5.127" x2="109" y2="3.5" width="0" layer="20" curve="-90"/>
+<wire x1="109" y1="3.5" x2="109" y2="1.5" width="0" layer="20"/>
+<wire x1="109" y1="1.5" x2="107.5" y2="0" width="0" layer="20" curve="-90"/>
+<wire x1="107.5" y1="0" x2="3.5" y2="0" width="0" layer="20"/>
 <text x="77.343" y="52.197" size="3.175" layer="26" rot="MR0" align="center">duckyPad Pro</text>
 <text x="77.343" y="43.815" size="2.1844" layer="26" rot="MR0" align="center">dekuNukem
 2024</text>
+<wire x1="105.5" y1="96" x2="109" y2="92.5" width="0" layer="20" curve="-90"/>
+<wire x1="109" y1="92.5" x2="109" y2="33.5" width="0" layer="20"/>
+<wire x1="109" y1="33.5" x2="107.5" y2="32" width="0" layer="20" curve="-90"/>
+<wire x1="107.5" y1="32" x2="101.5" y2="32" width="0" layer="20"/>
+<wire x1="101.5" y1="32" x2="100" y2="30.5" width="0" layer="20" curve="90"/>
+<wire x1="100" y1="30.5" x2="100" y2="22.5" width="0" layer="20"/>
+<wire x1="100" y1="22.5" x2="101.5" y2="21" width="0" layer="20" curve="90"/>
+<wire x1="101.5" y1="21" x2="107.5" y2="21" width="0" layer="20"/>
+<wire x1="107.5" y1="21" x2="109" y2="19.5" width="0" layer="20" curve="-90"/>
+<wire x1="109" y1="19.5" x2="107.5" y2="18.254" width="0" layer="20" curve="-90"/>
+<wire x1="107.5" y1="18.254" x2="105.5" y2="18.254" width="0" layer="20"/>
+<wire x1="105.5" y1="18.254" x2="104" y2="16.5" width="0" layer="20" curve="90"/>
 </plain>
 <attributes>
@@
 </autorouter>
 <elements>
-<element name="U$9" library="duckypad" package="M2_SCREW_FOOT" value="M2_SCREW_DEV" x="58.5" y="76.5" smashed="yes"/>
-<element name="U$10" library="duckypad" package="M2_SCREW_FOOT" value="M2_SCREW_DEV" x="92.75" y="7" smashed="yes"/>
-<element name="U$8" library="duckypad" package="M2_SCREW_FOOT" value="M2_SCREW_DEV" x="39.5" y="57.5" smashed="yes"/>
-<element name="U$12" library="duckypad" package="M2_SCREW_FOOT" value="M2_SCREW_DEV" x="39.5" y="38.5" smashed="yes"/>
-<element name="U$13" library="duckypad" package="M2_SCREW_FOOT" value="M2_SCREW_DEV" x="58.5" y="19.5" smashed="yes"/>
-<element name="U$17" library="duckypad" package="M2_SCREW_FOOT" value="M2_SCREW_DEV" x="100" y="76.5" smashed="yes"/>
-<element name="U$14" library="duckypad" package="M2_SCREW_FOOT" value="M2_SCREW_DEV" x="19.5" y="76.5" smashed="yes"/>
-<element name="U$22" library="duckypad" package="M2_SCREW_FOOT" value="M2_SCREW_DEV" x="19.5" y="19.5" smashed="yes"/>
+<element name="U$9" library="duckypad" package="M2_SCREW_FOOT" value="M2_SCREW_DEV" x="57.5" y="76.5" smashed="yes"/>
+<element name="U$10" library="duckypad" package="M2_SCREW_FOOT" value="M2_SCREW_DEV" x="91.75" y="7" smashed="yes"/>
+<element name="U$8" library="duckypad" package="M2_SCREW_FOOT" value="M2_SCREW_DEV" x="38.5" y="57.5" smashed="yes"/>
+<element name="U$12" library="duckypad" package="M2_SCREW_FOOT" value="M2_SCREW_DEV" x="38.5" y="38.5" smashed="yes"/>
+<element name="U$13" library="duckypad" package="M2_SCREW_FOOT" value="M2_SCREW_DEV" x="57.5" y="19.5" smashed="yes"/>
+<element name="U$17" library="duckypad" package="M2_SCREW_FOOT" value="M2_SCREW_DEV" x="99" y="76.5" smashed="yes"/>
+<element name="U$14" library="duckypad" package="M2_SCREW_FOOT" value="M2_SCREW_DEV" x="19" y="76.5" smashed="yes"/>
+<element name="U$22" library="duckypad" package="M2_SCREW_FOOT" value="M2_SCREW_DEV" x="19" y="19.5" smashed="yes"/>
 </elements>
 <signals>
