File: pcb/plate/duckypad.brd (EAGLE design)
At the start: 110 x 96 mm, 27 parts

Commit message: update plates
Parts:
- moved U$14 14.9 mm to (19.5, 76.5)
- moved U$22 14.9 mm to (19.5, 19.5)
- moved U$1 14.1 mm to (10.0, 10.0)
- moved U$10 14.1 mm to (67.0, 29.0)
- moved U$11 14.1 mm to (10.0, 48.0)
- moved U$12 14.1 mm to (38.5, 38.5)
- moved U$13 14.1 mm to (57.5, 19.5)
- moved U$15 14.1 mm to (29.0, 48.0)
- moved U$16 14.1 mm to (48.0, 48.0)
- moved U$17 14.1 mm to (99.0, 76.5)
- moved U$18 14.1 mm to (67.0, 48.0)
- moved U$19 14.1 mm to (10.0, 67.0)
- moved U$2 14.1 mm to (29.0, 10.0)
- moved U$20 14.1 mm to (10.0, 86.0)
- moved U$21 14.1 mm to (29.0, 67.0)
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Other:
- board size 110 x 96 mm -> 109 x 96 mm
- board text added: "big round corner 3.5mm"
