File: pcb/expansion/expansion.brd (EAGLE design)
At the start: 78 x 42 mm, 36 parts, among them IC3 STM32F042F4, J1 AUDIO_JACK_3.5MM_PTH, J2 AUDIO_JACK_3.5MM_PTH, J3 AUDIO_JACK_3.5MM_PTH, J4 AUDIO_JACK_3.5MM_PTH, J5 AUDIO_JACK_3.5MM_PTH, J6 AUDIO_JACK_3.5MM_PTH, SW3 324_SW, SW4 324_SW, U1 USBC_16P, U2 USBC_16P, U4 XC6206_DEV

Commit message: working on pcb
Parts:
- added U$10, U$11, U$8, U$9: M2.5HOLE, f1c100s:M2.5HOLE
- moved U4 145.9 mm to (14.0, 23.7), turned to 90 degrees
- moved U1 81.1 mm to (85.1, 21.0), turned to 90 degrees
- moved U2 70.5 mm to (3.81, 21.0), turned to 270 degrees
- moved IC3 6.94 mm to (38.1, 21.1), turned to 90 degrees
- moved JP1 6.15 mm to (25.1, 27.9)
- moved U$4 6.07 mm to (12.1, 33.0)
- moved U$1 6.07 mm to (12.1, 9.02)
- moved J4 6.02 mm to (25.0, 3.94)
- moved JP4 6.02 mm to (25.0, 14.0)
- moved J1 6.02 mm to (25.0, 38.0)
- moved U$7 6.01 mm to (64.0, 33.0)
- moved U$3 6.01 mm to (64.0, 9.02)
- moved U$5 5.97 mm to (38.0, 33.0)
- moved U$2 5.97 mm to (38.0, 9.02)
- moved J3 5.96 mm to (77.0, 3.94)
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Other:
- board size 78 x 42 mm -> 89 x 42 mm

Commit message: working on pcb
Parts:
- removed U$12: DG2204R-5.0-8DG2204-8, atx4vc:DG2204R-8
- added R10, R11, R12, R8, R9: 10K, joyAnalog:0805
- added R3, R7: 5.1K, joyAnalog:0805
- C2: value 1uF -> 100nF
- C3: value 2.2uF -> 1uF
- C4: value 2.2uF -> 100nF
- moved R1 155.7 mm to (5.08, 13.5), turned to 270 degrees
- moved R2 155.3 mm to (5.08, 28.6), turned to 90 degrees
- moved C1 146.5 mm to (13.1, 22.5), turned to 90 degrees
- moved R6 139.3 mm to (20.7, 28.8), turned to 270 degrees
- moved C2 120.4 mm to (32.6, 21.8), turned to 270 degrees
- moved U$6 115.9 mm to (39.6, 1.27)
- moved C3 111.5 mm to (19.8, 22.5), turned to 90 degrees
- moved SW3 93.2 mm to (50.9, 23.2)
- moved SW4 68.7 mm to (50.9, 19.1), turned to 180 degrees
- moved R5 58.4 mm to (56.8, 17.9), turned to 180 degrees
- moved C4 55.0 mm to (43.9, 21.7)
- moved U4 2.50 mm to (16.1, 22.5)
- moved U$1 1.14 mm to (13.2, 9.02)
- moved U$4 1.14 mm to (13.2, 33.0)
- moved JP3 1.09 mm to (76.1, 28.6)
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Connections:
- removed net PC_SYNC: J1.TIP, R6.1
- removed net UART2_TX: U$6.4
- new net N$1: R3.1, U1.A5
- new net N$2: R7.1, U1.B5
- new net N$3: J1.TIP, JP1.2, R6.1
- new net N$4: J5.TIP, JP2.2, R8.1
- new net N$6: J6.TIP, JP3.2, R9.1
- new net N$7: J4.TIP, JP4.2, R10.1
- new net N$8: J2.TIP, JP5.2, R11.1
- new net N$9: J3.TIP, JP6.2, R12.1
- net +3V3: now also JP1.1, JP2.1, JP3.1, JP4.1, JP5.1, JP6.1, R10.2, R11.2, R12.2, R8.2, R9.2
- net +5V: now also U1.A4B9, U1.B4A9
- net GND: now also J2.SLEEVE, J3.SLEEVE, J4.SLEEVE, J6.SLEEVE, JP1.3, JP2.3, JP3.3, JP4.3, JP5.3, R3.2, R7.2, U1.A1B12, U1.B11A12, U1.P$13, U1.P$14, U1.P$15, U1.P$16
- net U2RX: now also U1.A7, U1.B7
- net U2TX: now also U1.A6, U1.B6
Routing:
- net U2RX: track 0.00 -> 64.0 mm
- net U2TX: track 0.00 -> 45.4 mm
- net +3V3: track 0.00 -> 45.4 mm
- net USBDN/U1TX: track 0.00 -> 31.1 mm
- net USBDP/U1RX: track 0.00 -> 29.9 mm
- net SWDIO: track 0.00 -> 20.1 mm
- net SWCLK: track 0.00 -> 19.7 mm
- net BUTTON2: track 0.00 -> 15.0 mm
- net +5V: track 0.00 -> 13.8 mm, vias 0 -> 2
- net N$1: track 0.00 -> 8.49 mm
- net N$33: track 0.00 -> 7.85 mm
- net N$31: track 0.00 -> 7.40 mm
- net N$2: track 0.00 -> 7.26 mm
- net BUTTON1: track 0.00 -> 4.40 mm
Other:
- board size 89 x 42 mm -> 88 x 42 mm

Commit message: working on pcb
Connections:
- net GND: now also JP6.3
- net N$3: now also IC3.6
- net N$4: now also IC3.7
- net N$6: now also IC3.10
- net N$7: now also IC3.14
- net N$8: now also IC3.2
- net N$9: now also IC3.3
Routing:
- net N$7: track 0.00 -> 104.6 mm
- net N$9: track 0.00 -> 49.1 mm
- net N$6: track 0.00 -> 48.5 mm
- net N$3: track 0.00 -> 30.7 mm
- net N$4: track 0.00 -> 27.5 mm
- net N$8: track 0.00 -> 26.3 mm
- net BUTTON1: track 4.40 -> 22.6 mm
- net +3V3: track 45.4 -> 59.3 mm

Commit message: working on pcb
Parts:
- added LED2: (no value), adafruit:CHIP-LED0805
- added R13: 5.1K, SparkFun-Passives:0805
- added U$12, U$13: PINHD1X2, adafruit_changed:1X02
- moved R4 137.1 mm to (23.2, 23.4), turned to 270 degrees
- moved LED1 135.0 mm to (25.3, 21.5), turned to 180 degrees
- moved C3 2.11 mm to (18.7, 24.3)
- moved U4 2.11 mm to (15.0, 24.3)
- moved C1 2.11 mm to (11.9, 24.3)
Connections:
- new net N$10: LED2.A, R13.2
- net +3V3: now also R13.1, R4.1
- net GND: now also U$1.P$3, U$1.P$4, U$2.P$3, U$2.P$4, U$3.P$3, U$3.P$4, U$4.P$1, U$4.P$2, U$5.P$1, U$5.P$2, U$7.P$1, U$7.P$2; no longer R4.1
- net N$3: now also U$4.P$3, U$4.P$4
- net N$4: now also U$5.P$3, U$5.P$4
- net N$5: now also LED1.A; no longer LED1.C
- net N$6: now also U$7.P$3, U$7.P$4
- net N$7: now also U$1.P$1, U$1.P$2
- net N$8: now also U$2.P$1, U$2.P$2
- net N$9: now also U$3.P$1, U$3.P$2
- net U2RX: now also U$13.1
- net U2TX: now also U$13.2
- net USBDN/U1TX: now also LED1.C, U$12.2
- net USBDP/U1RX: now also LED2.C, U$12.1
Routing:
- net +3V3: track 59.3 -> 218.4 mm
- net +5V: track 13.8 -> 93.3 mm, vias 2 -> 4
- net N$9: track 49.1 -> 63.0 mm
- net N$4: track 27.5 -> 41.0 mm
- net N$6: track 48.5 -> 61.9 mm
- net N$3: track 30.7 -> 44.0 mm
- net N$8: track 26.3 -> 38.2 mm
- net N$7: track 104.6 -> 112.0 mm
- net N$10: track 0.00 -> 2.54 mm
- net N$5: track 0.00 -> 2.05 mm
- net U2TX: track 45.4 -> 47.1 mm
- net USBDP/U1RX: track 29.9 -> 31.2 mm

Commit message: working on pcb
Parts:
- added JP7: (no value), adafruit_changed:1X03-CLEANBIG
- moved C2 0.25 mm to (32.4, 21.8)
- moved R13 0.25 mm to (30.1, 21.8)
Connections:
- new net N$11: IC3.11, JP7.1
- new net N$12: IC3.12, JP7.2
- new net N$13: IC3.13, JP7.3
Routing:
- net N$13: track 0.00 -> 13.2 mm
- net N$12: track 0.00 -> 5.75 mm
- net N$3: track 44.0 -> 47.9 mm
- net N$11: track 0.00 -> 2.72 mm
- net N$7: track 112.0 -> 109.6 mm
- net +3V3: track 218.4 -> 219.0 mm

Commit message: working on pcb
Parts:
- added LED3: (no value), adafruit:CHIP-LED0805
- added R14: 5.1K, SparkFun-Passives:0805
- JP7: device adafruit_changed:1X03-CLEANBIG -> adafruit_changed:1X01-CLEANBIG
- moved JP7 2.92 mm to (33.1, 24.9), turned to 0 degrees
Connections:
- removed net N$13 (its old number): IC3.13, JP7.3
- new net N$11: LED3.C, R14.2
- new net N$14: IC3.12, U$6.4
- net GND: now also R14.1
- net N$12: now also IC3.13, LED3.A; no longer IC3.12, JP7.2
Routing:
- net N$14: track 0.00 -> 56.2 mm, vias 0 -> 1
- net N$13 (its old number): track 13.2 -> 0.00 mm
- net +3V3: track 219.0 -> 224.1 mm
- net N$11: track 0.00 -> 1.61 mm
- net N$7: track 109.6 -> 110.8 mm
Other:
- board text added: "1"
- board text added: "3"
- board text added: "4"
- board text added: "6"
- board text added: "DFU"
- board text added: "U1RX"
- board text added: "U1TX"
- board text added: "U2RX"
- board text added: "U2TX"
- board text removed: "USER"

Commit message: working on pcb
Parts:
- moved U$12 4.06 mm to (21.2, 19.8)
- moved U$13 2.16 mm to (62.9, 22.2)
Routing:
- net N$14: track 56.2 -> 54.2 mm
Other:
- board text added: "3V"
- board text added: "S2"
- board text added: "S3"
- board text added: "S4"
- board text added: "S5"
- board text added: "S6"
- board text added: "TOWARDS DUCKYPAD"

Commit message: working on pcb
Parts:
- moved R5 1.59 mm to (56.0, 16.5), turned to 90 degrees
Other:
- outline, holes or cut-outs redrawn
- board text added: "DUCKY PAD <<--"
- board text added: "U1R"
- board text added: "U1T"
- board text removed: "TOWARDS DUCKYPAD"
- board text removed: "U1RX"
- board text removed: "U1TX"
Changed lines of the file:
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@@
 <layer number="14" name="Route14" color="22" fill="1" visible="no" active="no"/>
 <layer number="15" name="Route15" color="23" fill="1" visible="no" active="no"/>
-<layer number="16" name="Bottom" color="1" fill="1" visible="no" active="yes"/>
+<layer number="16" name="Bottom" color="1" fill="1" visible="yes" active="yes"/>
 <layer number="17" name="Pads" color="2" fill="1" visible="yes" active="yes"/>
 <layer number="18" name="Vias" color="2" fill="1" visible="yes" active="yes"/>
@@
 <layer number="20" name="Dimension" color="24" fill="1" visible="yes" active="yes"/>
 <layer number="21" name="tPlace" color="7" fill="1" visible="yes" active="yes"/>
-<layer number="22" name="bPlace" color="7" fill="1" visible="no" active="yes"/>
+<layer number="22" name="bPlace" color="7" fill="1" visible="yes" active="yes"/>
 <layer number="23" name="tOrigins" color="15" fill="1" visible="yes" active="yes"/>
-<layer number="24" name="bOrigins" color="15" fill="1" visible="no" active="yes"/>
+<layer number="24" name="bOrigins" color="15" fill="1" visible="yes" active="yes"/>
 <layer number="25" name="tNames" color="7" fill="1" visible="yes" active="yes"/>
-<layer number="26" name="bNames" color="7" fill="1" visible="no" active="yes"/>
-<layer number="27" name="tValues" color="7" fill="1" visible="no" active="yes"/>
-<layer number="28" name="bValues" color="7" fill="1" visible="no" active="yes"/>
+<layer number="26" name="bNames" color="7" fill="1" visible="yes" active="yes"/>
+<layer number="27" name="tValues" color="7" fill="1" visible="yes" active="yes"/>
+<layer number="28" name="bValues" color="7" fill="1" visible="yes" active="yes"/>
 <layer number="29" name="tStop" color="7" fill="3" visible="no" active="yes"/>
 <layer number="30" name="bStop" color="7" fill="6" visible="no" active="yes"/>
@@
 <layer number="38" name="bTest" color="7" fill="1" visible="no" active="yes"/>
 <layer number="39" name="tKeepout" color="4" fill="11" visible="yes" active="yes"/>
-<layer number="40" name="bKeepout" color="1" fill="11" visible="no" active="yes"/>
+<layer number="40" name="bKeepout" color="1" fill="11" visible="yes" active="yes"/>
 <layer number="41" name="tRestrict" color="4" fill="10" visible="yes" active="yes"/>
-<layer number="42" name="bRestrict" color="1" fill="10" visible="no" active="yes"/>
+<layer number="42" name="bRestrict" color="1" fill="10" visible="yes" active="yes"/>
 <layer number="43" name="vRestrict" color="2" fill="10" visible="no" active="yes"/>
 <layer number="44" name="Drills" color="7" fill="1" visible="yes" active="yes"/>
@@
 <layer number="50" name="dxf" color="7" fill="1" visible="no" active="no"/>
 <layer number="51" name="tDocu" color="7" fill="1" visible="yes" active="yes"/>
-<layer number="52" name="bDocu" color="7" fill="1" visible="no" active="yes"/>
+<layer number="52" name="bDocu" color="7" fill="1" visible="yes" active="yes"/>
 <layer number="53" name="tGND_GNDA" color="7" fill="1" visible="no" active="no"/>
 <layer number="54" name="bGND_GNDA" color="7" fill="1" visible="no" active="no"/>
@@
 <text x="156.4448" y="25.3036" size="1.27" layer="25" rot="R180" align="center">G</text>
 <text x="146.3174" y="24.3448" size="1.27" layer="25" rot="R270" align="center">3V3</text>
-<text x="45.2952" y="19.0434" size="1.9304" layer="25" align="center">DFU</text>
-<text x="58.1222" y="22.9804" size="1.9304" layer="25" align="center">RESET</text>
+<text x="56.7252" y="19.0434" size="1.9304" layer="25" align="center">DFU</text>
+<text x="58.1222" y="23.1074" size="1.9304" layer="25" align="center">RESET</text>
 <text x="157.639" y="17.792" size="1.27" layer="25" rot="R90" align="center">PC</text>
 <text x="157.639" y="15.125" size="1.27" layer="25" align="center">G</text>
 <text x="146.6562" y="43.3924" size="2.1082" layer="26" rot="MR0" align="center">PulseHPT.com
 dekuNukem 2023</text>
-<wire x1="0.5" y1="42" x2="88.5" y2="42" width="0" layer="20"/>
-<wire x1="88.5" y1="42" x2="88.5" y2="0" width="0" layer="20"/>
-<wire x1="88.5" y1="0" x2="0.5" y2="0" width="0" layer="20"/>
-<wire x1="0.5" y1="0" x2="0.5" y2="42" width="0" layer="20"/>
-<text x="62.9042" y="25.1594" size="1.016" layer="51" align="center">U2RX</text>
-<text x="62.9042" y="19.3174" size="1.016" layer="51" align="center">U2TX</text>
-<text x="20.9942" y="22.6194" size="1.016" layer="51" align="center">U1TX</text>
-<text x="24.1692" y="18.4284" size="1.016" layer="51" align="center">U1RX</text>
+<wire x1="3" y1="42" x2="86" y2="42" width="0" layer="20"/>
+<wire x1="86" y1="42" x2="88.5" y2="39.5" width="0" layer="20" curve="-90"/>
+<wire x1="88.5" y1="39.5" x2="88.5" y2="2.5" width="0" layer="20"/>
+<wire x1="88.5" y1="2.5" x2="86" y2="0" width="0" layer="20" curve="-90"/>
+<wire x1="86" y1="0" x2="3" y2="0" width="0" layer="20"/>
+<wire x1="3" y1="0" x2="0.5" y2="2.5" width="0" layer="20" curve="-90"/>
+<wire x1="0.5" y1="2.5" x2="0.5" y2="39.5" width="0" layer="20"/>
+<wire x1="0.5" y1="39.5" x2="3" y2="42" width="0" layer="20" curve="-90"/>
+<text x="62.9042" y="25.1594" size="1.016" layer="25" align="center">U2RX</text>
+<text x="62.9042" y="19.3174" size="1.016" layer="25" align="center">U2TX</text>
+<text x="20.9942" y="22.7464" size="1.27" layer="25" align="center">U1T</text>
+<text x="23.9152" y="18.4284" size="1.27" layer="25" align="center">U1R</text>
 <text x="3.6638" y="33.0506" size="5.08" layer="25" rot="R180" align="center">1</text>
 <text x="85.5788" y="33.1776" size="5.08" layer="25" rot="R180" align="center">3</text>
@@
 <text x="50.9662" y="26.1754" size="1.27" layer="25" align="center">S2</text>
 <text x="53.4478" y="15.9056" size="1.27" layer="25" rot="R180" align="center">G</text>
-<text x="42.2472" y="51.8094" size="1.6764" layer="25" align="center">TOWARDS
-DUCKYPAD</text>
+<text x="15.1568" y="19.3106" size="1.9304" layer="25" distance="15" rot="R180" align="center">DUCKY
+PAD
+&lt;&lt;--</text>
+<text x="71.7988" y="20.5806" size="2.1844" layer="25" distance="15" rot="R180" align="center">DUCKY
+PAD
+&lt;&lt;--</text>
 </plain>
 <attributes>
@@
 </element>
 <element name="C1" library="clock" package="0805" value="1uF" x="11.938" y="24.257" smashed="yes" rot="R90">
-<attribute name="NAME" x="11.4935" y="22.5298" size="0.8128" layer="25" rot="R270"/>
+<attribute name="NAME" x="10.2235" y="25.3238" size="0.8128" layer="25" rot="R270"/>
 </element>
 <element name="IC3" library="tx" package="TSSOP20" value="STM32F042F4" x="38.108" y="21.12" smashed="yes" rot="R90"/>
@@
 <attribute name="NAME" x="22.8981" y="21.6916" size="0.8128" layer="25" rot="R270"/>
 </element>
-<element name="R5" library="joyAnalog" package="0805" value="10K" x="56.769" y="17.907" smashed="yes" rot="R180">
-<attribute name="NAME" x="58.4416" y="17.4155" size="0.8128" layer="25"/>
+<element name="R5" library="joyAnalog" package="0805" value="10K" x="56.007" y="16.51" smashed="yes" rot="R90">
+<attribute name="NAME" x="55.5155" y="14.8374" size="0.8128" layer="25" rot="R270"/>
 </element>
 <element name="U4" library="3pos_slide_switch" package="SOT23R_INFINEON" value="XC6206_DEV" x="14.986" y="24.257" smashed="yes" rot="R90"/>
@@
 </element>
 <element name="R11" library="joyAnalog" package="0805" value="10K" x="56.007" y="13.462" smashed="yes" rot="R90">
-<attribute name="NAME" x="56.769" y="15.8115" size="0.8128" layer="25" rot="R180"/>
+<attribute name="NAME" x="57.7215" y="14.097" size="0.8128" layer="25" rot="R270"/>
 </element>
 <element name="R12" library="joyAnalog" package="0805" value="10K" x="81.407" y="12.954" smashed="yes" rot="R90">
@@
 <wire x1="48.457" y1="18.195" x2="48.727" y2="17.925" width="0.3048" layer="1"/>
 <wire x1="48.727" y1="17.925" x2="53.127" y2="17.925" width="1.016" layer="1"/>
-<wire x1="53.127" y1="17.925" x2="55.851" y2="17.925" width="0.3048" layer="1"/>
-<wire x1="55.851" y1="17.925" x2="55.869" y2="17.907" width="0.3048" layer="1"/>
+<wire x1="53.127" y1="17.925" x2="55.492" y2="17.925" width="0.2032" layer="1"/>
+<wire x1="55.492" y1="17.925" x2="56.007" y2="17.41" width="0.2032" layer="1"/>
 </signal>
 <signal name="SWCLK">
