File: pcb/expansion/expansion.sch (EAGLE design)
At the start: 36 parts, among them IC3 STM32F042F4, J1 AUDIO_JACK_3.5MM_PTH, J2 AUDIO_JACK_3.5MM_PTH, J3 AUDIO_JACK_3.5MM_PTH, J4 AUDIO_JACK_3.5MM_PTH, J5 AUDIO_JACK_3.5MM_PTH, J6 AUDIO_JACK_3.5MM_PTH, SW3 324_SW, SW4 324_SW, U1 USBC_16P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

Commit message: working on pcb
Parts:
- added U$10, U$11, U$8, U$9: M2.5HOLE, f1c100s:M2.5HOLE
Changed lines of the file:
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@@
 <part name="JP5" library="pinhead" library_urn="urn:adsk.eagle:library:325" deviceset="PINHD-1X3" device="" package3d_urn="urn:adsk.eagle:package:22458/2"/>
 <part name="JP6" library="pinhead" library_urn="urn:adsk.eagle:library:325" deviceset="PINHD-1X3" device="" package3d_urn="urn:adsk.eagle:package:22458/2"/>
+<part name="U$8" library="f1c100s" deviceset="M2.5HOLE" device=""/>
+<part name="U$9" library="f1c100s" deviceset="M2.5HOLE" device=""/>
+<part name="U$10" library="f1c100s" deviceset="M2.5HOLE" device=""/>
+<part name="U$11" library="f1c100s" deviceset="M2.5HOLE" device=""/>
 </parts>
 <sheets>
@@
 <attribute name="VALUE" x="168.91" y="-101.6" size="1.778" layer="96"/>
 </instance>
+<instance part="U$8" gate="G$1" x="238.76" y="-71.12" smashed="yes"/>
+<instance part="U$9" gate="G$1" x="238.76" y="-86.36" smashed="yes"/>
+<instance part="U$10" gate="G$1" x="297.18" y="-71.12" smashed="yes"/>
+<instance part="U$11" gate="G$1" x="297.18" y="-86.36" smashed="yes"/>
 </instances>
 <busses>

Commit message: working on pcb
Parts:
- removed U$12: DG2204R-5.0-8DG2204-8, atx4vc:DG2204R-5.0-8DG2204-8
- added R10, R11, R12, R8, R9: 10K, joyAnalog:RESISTOR0805-RES
- added R3, R7: 5.1K, joyAnalog:RESISTOR0805-RES
- C2: value 1uF -> 100nF
- C3: value 2.2uF -> 1uF
- C4: value 2.2uF -> 100nF
Connections:
- removed net PC_SYNC: J1.TIP, R6.1
- removed net UART2_TX: U$6.4
- new net N$1: R3.1, U1.CC1
- new net N$2: R7.1, U1.CC2
- new net N$3: J1.TIP, JP1.2, R6.1
- new net N$4: J5.TIP, JP2.2, R8.1
- new net N$6: J6.TIP, JP3.2, R9.1
- new net N$7: J4.TIP, JP4.2, R10.1
- new net N$8: J2.TIP, JP5.2, R11.1
- new net N$9: J3.TIP, JP6.2, R12.1
- net +3V3: now also JP1.1, JP2.1, JP3.1, JP4.1, JP5.1, JP6.1, R10.2, R11.2, R12.2, R8.2, R9.2
- net +5V: now also U1.VBUS
- net GND: now also J2.SLEEVE, J3.SLEEVE, J4.SLEEVE, J6.SLEEVE, JP1.3, JP2.3, JP3.3, JP4.3, JP5.3, R3.2, R7.2, U1.GND
- net U2RX: now also U1.DN1, U1.DN2
- net U2TX: now also U1.DP1, U1.DP2
Other:
- moved on the sheet: C2, C3, C4, J1, J2, J3, J4, J5, J6, JP1, JP2, JP3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

Commit message: working on pcb
Connections:
- net GND: now also JP6.3
- net N$3: now also IC3.PA0
- net N$4: now also IC3.PA1
- net N$6: now also IC3.PA4
- net N$7: now also IC3.PB1
- net N$8: now also IC3.PF0/OSC_IN
- net N$9: now also IC3.PF1/OSC_OUT
Changed lines of the file:
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@@
 <part name="LED1" library="adafruit" deviceset="LED" device="CHIP-LED0805"/>
 <part name="R4" library="SparkFun-Passives" deviceset="RESISTOR" device="0805-RES" value="5.1K"/>
-<part name="+3V2" library="supply1" library_urn="urn:adsk.eagle:library:371" deviceset="+3V3" device=""/>
 <part name="R5" library="joyAnalog" deviceset="RESISTOR" device="0805-RES" value="10K"/>
 <part name="GND10" library="supply1" deviceset="GND" device=""/>
@@
 <part name="R12" library="joyAnalog" deviceset="RESISTOR" device="0805-RES" value="10K"/>
 <part name="GND19" library="supply1" deviceset="GND" device=""/>
+<part name="+3V2" library="supply1" library_urn="urn:adsk.eagle:library:371" deviceset="+3V3" device=""/>
 </parts>
 <sheets>
@@
 <attribute name="NAME" x="-6.35" y="-47.2186" size="1.778" layer="95" rot="R180"/>
 <attribute name="VALUE" x="-6.35" y="-42.418" size="1.778" layer="96" rot="R180"/>
-</instance>
-<instance part="+3V2" gate="G$1" x="93.98" y="25.4" smashed="yes" rot="MR0">
-<attribute name="VALUE" x="96.52" y="20.32" size="1.778" layer="96" rot="MR90"/>
 </instance>
 <instance part="R5" gate="G$1" x="76.2" y="12.7" smashed="yes" rot="MR90">
@@
 <attribute name="VALUE" x="187.96" y="-99.06" size="1.778" layer="96" rot="MR0"/>
 </instance>
+<instance part="+3V2" gate="G$1" x="93.98" y="20.32" smashed="yes" rot="MR0">
+<attribute name="VALUE" x="88.9" y="15.24" size="1.778" layer="96" rot="MR90"/>
+</instance>
 </instances>
 <busses>
@@
 <wire x1="180.34" y1="-93.98" x2="185.42" y2="-93.98" width="0.1524" layer="91"/>
 <pinref part="J3" gate="G$1" pin="SLEEVE"/>
-<wire x1="180.34" y1="-93.98" x2="180.34" y2="-119.38" width="0.1524" layer="91"/>
+<wire x1="180.34" y1="-93.98" x2="180.34" y2="-104.14" width="0.1524" layer="91"/>
+<pinref part="JP6" gate="A" pin="3"/>
+<wire x1="180.34" y1="-104.14" x2="180.34" y2="-119.38" width="0.1524" layer="91"/>
+<wire x1="172.72" y1="-104.14" x2="180.34" y2="-104.14" width="0.1524" layer="91"/>
+<junction x="180.34" y="-104.14"/>
 </segment>
 </net>
@@
 </segment>
 <segment>
-<pinref part="SW4" gate="G$1" pin="1"/>
-<pinref part="SW4" gate="G$1" pin="4"/>
-<wire x1="93.98" y1="22.86" x2="93.98" y2="-12.7" width="0.1524" layer="91"/>
-<pinref part="+3V2" gate="G$1" pin="+3V3"/>
-<junction x="93.98" y="22.86"/>
-<wire x1="93.98" y1="22.86" x2="93.98" y2="17.78" width="0.1524" layer="91"/>
-</segment>
-<segment>
 <pinref part="C4" gate="G$1" pin="2"/>
 <pinref part="+3V3" gate="G$1" pin="+3V3"/>
@@
 <junction x="167.64" y="-86.36"/>
 <pinref part="JP6" gate="A" pin="1"/>
+</segment>
+<segment>
+<pinref part="SW4" gate="G$1" pin="1"/>
+<pinref part="SW4" gate="G$1" pin="4"/>
+<wire x1="93.98" y1="17.78" x2="93.98" y2="-12.7" width="0.1524" layer="91"/>
+<pinref part="+3V2" gate="G$1" pin="+3V3"/>
+<junction x="93.98" y="17.78"/>
 </segment>
 </net>
@@
 <pinref part="J1" gate="G$1" pin="TIP"/>
 <pinref part="JP1" gate="A" pin="2"/>
-<wire x1="-40.64" y1="-111.76" x2="-40.64" y2="-104.14" width="0.1524" layer="91"/>
+<wire x1="-40.64" y1="-111.76" x2="-40.64" y2="-109.22" width="0.1524" layer="91"/>
 <pinref part="R6" gate="G$1" pin="1"/>
+<wire x1="-40.64" y1="-109.22" x2="-40.64" y2="-104.14" width="0.1524" layer="91"/>
 <wire x1="-40.64" y1="-96.52" x2="-40.64" y2="-104.14" width="0.1524" layer="91"/>
 <junction x="-40.64" y="-104.14"/>
+<pinref part="IC3" gate="G$1" pin="PA0"/>
+<wire x1="-17.78" y1="40.64" x2="-58.42" y2="40.64" width="0.1524" layer="91"/>
+<wire x1="-58.42" y1="40.64" x2="-58.42" y2="-109.22" width="0.1524" layer="91"/>
+<wire x1="-58.42" y1="-109.22" x2="-40.64" y2="-109.22" width="0.1524" layer="91"/>
+<junction x="-40.64" y="-109.22"/>
 </segment>
 </net>
@@
 <pinref part="JP2" gate="A" pin="2"/>
 <pinref part="J5" gate="G$1" pin="TIP"/>
-<wire x1="-5.08" y1="-106.68" x2="-5.08" y2="-116.84" width="0.1524" layer="91"/>
+<wire x1="-5.08" y1="-106.68" x2="-5.08" y2="-114.3" width="0.1524" layer="91"/>
 <junction x="-5.08" y="-106.68"/>
+<pinref part="IC3" gate="G$1" pin="PA1"/>
+<wire x1="-5.08" y1="-114.3" x2="-5.08" y2="-116.84" width="0.1524" layer="91"/>
+<wire x1="-17.78" y1="38.1" x2="-55.88" y2="38.1" width="0.1524" layer="91"/>
+<wire x1="-55.88" y1="38.1" x2="-55.88" y2="-63.5" width="0.1524" layer="91"/>
+<wire x1="-55.88" y1="-63.5" x2="-12.7" y2="-63.5" width="0.1524" layer="91"/>
+<wire x1="-12.7" y1="-63.5" x2="-12.7" y2="-114.3" width="0.1524" layer="91"/>
+<wire x1="-12.7" y1="-114.3" x2="-5.08" y2="-114.3" width="0.1524" layer="91"/>
+<junction x="-5.08" y="-114.3"/>
 </segment>
 </net>
@@
 <pinref part="JP3" gate="A" pin="2"/>
 <pinref part="J6" gate="G$1" pin="TIP"/>
-<wire x1="45.72" y1="-116.84" x2="45.72" y2="-104.14" width="0.1524" layer="91"/>
+<wire x1="45.72" y1="-116.84" x2="45.72" y2="-111.76" width="0.1524" layer="91"/>
 <junction x="45.72" y="-104.14"/>
+<pinref part="IC3" gate="G$1" pin="PA4"/>
+<wire x1="45.72" y1="-111.76" x2="45.72" y2="-104.14" width="0.1524" layer="91"/>
+<wire x1="-17.78" y1="30.48" x2="-50.8" y2="30.48" width="0.1524" layer="91"/>
+<wire x1="-50.8" y1="30.48" x2="-50.8" y2="-60.96" width="0.1524" layer="91"/>
+<wire x1="-50.8" y1="-60.96" x2="30.48" y2="-60.96" width="0.1524" layer="91"/>
+<wire x1="30.48" y1="-60.96" x2="30.48" y2="-111.76" width="0.1524" layer="91"/>
+<wire x1="30.48" y1="-111.76" x2="45.72" y2="-111.76" width="0.1524" layer="91"/>
+<junction x="45.72" y="-111.76"/>
 </segment>
 </net>
@@
 <pinref part="JP4" gate="A" pin="2"/>
 <pinref part="J4" gate="G$1" pin="TIP"/>
-<wire x1="86.36" y1="-104.14" x2="86.36" y2="-116.84" width="0.1524" layer="91"/>
+<wire x1="86.36" y1="-104.14" x2="86.36" y2="-111.76" width="0.1524" layer="91"/>
 <junction x="86.36" y="-104.14"/>
+<pinref part="IC3" gate="G$1" pin="PB1"/>
+<wire x1="86.36" y1="-111.76" x2="86.36" y2="-116.84" width="0.1524" layer="91"/>
+<wire x1="-17.78" y1="7.62" x2="-63.5" y2="7.62" width="0.1524" layer="91"/>
+<wire x1="-63.5" y1="7.62" x2="-63.5" y2="-149.86" width="0.1524" layer="91"/>
+<wire x1="-63.5" y1="-149.86" x2="78.74" y2="-149.86" width="0.1524" layer="91"/>
+<wire x1="78.74" y1="-149.86" x2="78.74" y2="-111.76" width="0.1524" layer="91"/>
+<wire x1="78.74" y1="-111.76" x2="86.36" y2="-111.76" width="0.1524" layer="91"/>
+<junction x="86.36" y="-111.76"/>
 </segment>
 </net>
@@
 <pinref part="JP5" gate="A" pin="2"/>
 <pinref part="J2" gate="G$1" pin="TIP"/>
-<wire x1="134.62" y1="-104.14" x2="134.62" y2="-119.38" width="0.1524" layer="91"/>
+<wire x1="134.62" y1="-104.14" x2="134.62" y2="-114.3" width="0.1524" layer="91"/>
 <junction x="134.62" y="-104.14"/>
+<pinref part="IC3" gate="G$1" pin="PF0/OSC_IN"/>
+<wire x1="134.62" y1="-114.3" x2="134.62" y2="-119.38" width="0.1524" layer="91"/>
+<wire x1="20.32" y1="27.94" x2="124.46" y2="27.94" width="0.1524" layer="91"/>
+<wire x1="124.46" y1="27.94" x2="124.46" y2="-114.3" width="0.1524" layer="91"/>
+<wire x1="124.46" y1="-114.3" x2="134.62" y2="-114.3" width="0.1524" layer="91"/>
+<junction x="134.62" y="-114.3"/>
 </segment>
 </net>
@@
 <pinref part="JP6" gate="A" pin="2"/>
 <pinref part="J3" gate="G$1" pin="TIP"/>
-<wire x1="170.18" y1="-104.14" x2="170.18" y2="-119.38" width="0.1524" layer="91"/>
+<wire x1="170.18" y1="-104.14" x2="170.18" y2="-111.76" width="0.1524" layer="91"/>
 <junction x="170.18" y="-104.14"/>
-</segment>
-</net>
+<pinref part="IC3" gate="G$1" pin="PF1/OSC_OUT"/>
+<wire x1="170.18" y1="-111.76" x2="170.18" y2="-119.38" width="0.1524" layer="91"/>
+<wire x1="20.32" y1="25.4" x2="162.56" y2="25.4" width="0.1524" layer="91"/>
+<wire x1="162.56" y1="25.4" x2="162.56" y2="-111.76" width="0.1524" layer="91"/>
+<wire x1="162.56" y1="-111.76" x2="170.18" y2="-111.76" width="0.1524" layer="91"/>
+<junction x="170.18" y="-111.76"/>
+</segment>
+</net>

Commit message: working on pcb
Parts:
- added LED2: (no value), adafruit:LEDCHIP-LED0805
- added R13: 5.1K, SparkFun-Passives:RESISTOR0805-RES
- added U$12, U$13: PINHD1X2, adafruit_changed:PINHD1X2
Connections:
- new net N$10: LED2.A, R13.2
- net +3V3: now also R13.1, R4.1
- net GND: now also U$1.P$2, U$2.P$2, U$3.P$2, U$4.P$1, U$5.P$1, U$7.P$1; no longer R4.1
- net N$3: now also U$4.P$2
- net N$4: now also U$5.P$2
- net N$5: now also LED1.A; no longer LED1.C
- net N$6: now also U$7.P$2
- net N$7: now also U$1.P$1
- net N$8: now also U$2.P$1
- net N$9: now also U$3.P$1
- net U2RX: now also U$13.1
- net U2TX: now also U$13.2
- net USBDN/U1TX: now also LED1.C, U$12.2
- net USBDP/U1RX: now also LED2.C, U$12.1
Other:
- moved on the sheet: LED1, R4

Commit message: working on pcb
Parts:
- added JP7: (no value), adafruit_changed:PINHD-1X3CB
Connections:
- new net N$11: IC3.PA5, JP7.1
- new net N$12: IC3.PA6, JP7.2
- new net N$13: IC3.PA7, JP7.3
Changed lines of the file:
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@@
 <part name="U$12" library="adafruit_changed" deviceset="PINHD1X2" device=""/>
 <part name="U$13" library="adafruit_changed" deviceset="PINHD1X2" device=""/>
+<part name="JP7" library="adafruit_changed" deviceset="PINHD-1X3" device="CB"/>
 </parts>
 <sheets>
@@
 <attribute name="NAME" x="-44.45" y="29.845" size="1.778" layer="95" rot="R180"/>
 <attribute name="VALUE" x="-44.45" y="40.64" size="1.778" layer="96" rot="R180"/>
+</instance>
+<instance part="JP7" gate="A" x="0" y="25.4" smashed="yes">
+<attribute name="NAME" x="-6.35" y="31.115" size="1.778" layer="95"/>
+<attribute name="VALUE" x="-6.35" y="17.78" size="1.778" layer="96"/>
 </instance>
 </instances>
@@
 </segment>
 </net>
+<net name="N$11" class="0">
+<segment>
+<pinref part="IC3" gate="G$1" pin="PA5"/>
+<pinref part="JP7" gate="A" pin="1"/>
+<wire x1="-17.78" y1="27.94" x2="-2.54" y2="27.94" width="0.1524" layer="91"/>
+</segment>
+</net>
+<net name="N$12" class="0">
+<segment>
+<pinref part="JP7" gate="A" pin="2"/>
+<pinref part="IC3" gate="G$1" pin="PA6"/>
+<wire x1="-2.54" y1="25.4" x2="-17.78" y2="25.4" width="0.1524" layer="91"/>
+</segment>
+</net>
+<net name="N$13" class="0">
+<segment>
+<pinref part="IC3" gate="G$1" pin="PA7"/>
+<pinref part="JP7" gate="A" pin="3"/>
+<wire x1="-17.78" y1="22.86" x2="-2.54" y2="22.86" width="0.1524" layer="91"/>
+</segment>
+</net>

Commit message: working on pcb
Parts:
- added LED3: (no value), adafruit:LEDCHIP-LED0805
- added R14: 5.1K, SparkFun-Passives:RESISTOR0805-RES
- JP7: device adafruit_changed:PINHD-1X3CB -> adafruit_changed:PINHD-1X1CB
Connections:
- removed net N$13 (its old number): IC3.PA7, JP7.3
- new net N$11: LED3.C, R14.2
- new net N$14: IC3.PA6, U$6.4
- net GND: now also R14.1
- net N$12: now also IC3.PA7, LED3.A; no longer IC3.PA6, JP7.2
Changed lines of the file:
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@@
 <part name="U$12" library="adafruit_changed" deviceset="PINHD1X2" device=""/>
 <part name="U$13" library="adafruit_changed" deviceset="PINHD1X2" device=""/>
-<part name="JP7" library="adafruit_changed" deviceset="PINHD-1X3" device="CB"/>
+<part name="LED3" library="adafruit" deviceset="LED" device="CHIP-LED0805"/>
+<part name="R14" library="SparkFun-Passives" deviceset="RESISTOR" device="0805-RES" value="5.1K"/>
+<part name="GND18" library="supply1" deviceset="GND" device=""/>
+<part name="JP7" library="adafruit_changed" deviceset="PINHD-1X1" device="CB"/>
 </parts>
 <sheets>
@@
 <attribute name="VALUE" x="-44.45" y="40.64" size="1.778" layer="96" rot="R180"/>
 </instance>
-<instance part="JP7" gate="A" x="0" y="25.4" smashed="yes">
-<attribute name="NAME" x="-6.35" y="31.115" size="1.778" layer="95"/>
-<attribute name="VALUE" x="-6.35" y="17.78" size="1.778" layer="96"/>
+<instance part="LED3" gate="G$1" x="-2.54" y="-5.08" smashed="yes" rot="R90">
+<attribute name="NAME" x="2.032" y="-1.524" size="1.778" layer="95" rot="R180"/>
+<attribute name="VALUE" x="2.032" y="0.635" size="1.778" layer="96" rot="R180"/>
+</instance>
+<instance part="R14" gate="G$1" x="10.16" y="-5.08" smashed="yes" rot="R180">
+<attribute name="NAME" x="13.97" y="-6.5786" size="1.778" layer="95" rot="R180"/>
+<attribute name="VALUE" x="13.97" y="-1.778" size="1.778" layer="96" rot="R180"/>
+</instance>
+<instance part="GND18" gate="1" x="20.32" y="-7.62" smashed="yes" rot="MR0">
+<attribute name="VALUE" x="22.86" y="-10.16" size="1.778" layer="96" rot="MR0"/>
+</instance>
+<instance part="JP7" gate="G$1" x="-30.48" y="27.94" smashed="yes" rot="R180">
+<attribute name="NAME" x="-24.13" y="24.765" size="1.778" layer="95" rot="R180"/>
+<attribute name="VALUE" x="-24.13" y="33.02" size="1.778" layer="96" rot="R180"/>
 </instance>
 </instances>
@@
 <pinref part="GND21" gate="1" pin="GND"/>
 <wire x1="157.48" y1="-139.7" x2="152.4" y2="-139.7" width="0.1524" layer="91"/>
+</segment>
+<segment>
+<pinref part="GND18" gate="1" pin="GND"/>
+<pinref part="R14" gate="G$1" pin="1"/>
+<wire x1="20.32" y1="-5.08" x2="15.24" y2="-5.08" width="0.1524" layer="91"/>
 </segment>
 </net>
@@
 <net name="N$11" class="0">
 <segment>
+<pinref part="LED3" gate="G$1" pin="C"/>
+<pinref part="R14" gate="G$1" pin="2"/>
+<wire x1="5.08" y1="-5.08" x2="2.54" y2="-5.08" width="0.1524" layer="91"/>
+</segment>
+</net>
+<net name="N$12" class="0">
+<segment>
+<pinref part="IC3" gate="G$1" pin="PA7"/>
+<pinref part="LED3" gate="G$1" pin="A"/>
+<wire x1="-17.78" y1="22.86" x2="-5.08" y2="22.86" width="0.1524" layer="91"/>
+<wire x1="-5.08" y1="22.86" x2="-5.08" y2="-5.08" width="0.1524" layer="91"/>
+</segment>
+</net>
+<net name="N$13" class="0">
+<segment>
 <pinref part="IC3" gate="G$1" pin="PA5"/>
-<pinref part="JP7" gate="A" pin="1"/>
-<wire x1="-17.78" y1="27.94" x2="-2.54" y2="27.94" width="0.1524" layer="91"/>
-</segment>
-</net>
-<net name="N$12" class="0">
-<segment>
-<pinref part="JP7" gate="A" pin="2"/>
+<pinref part="JP7" gate="G$1" pin="1"/>
+<wire x1="-17.78" y1="27.94" x2="-27.94" y2="27.94" width="0.1524" layer="91"/>
+</segment>
+</net>
+<net name="N$14" class="0">
+<segment>
 <pinref part="IC3" gate="G$1" pin="PA6"/>
-<wire x1="-2.54" y1="25.4" x2="-17.78" y2="25.4" width="0.1524" layer="91"/>
-</segment>
-</net>
-<net name="N$13" class="0">
-<segment>
-<pinref part="IC3" gate="G$1" pin="PA7"/>
-<pinref part="JP7" gate="A" pin="3"/>
-<wire x1="-17.78" y1="22.86" x2="-2.54" y2="22.86" width="0.1524" layer="91"/>
-</segment>
-</net>
+<wire x1="-17.78" y1="25.4" x2="-73.66" y2="25.4" width="0.1524" layer="91"/>
+<pinref part="U$6" gate="G$1" pin="4"/>
+<wire x1="-73.66" y1="25.4" x2="-73.66" y2="30.48" width="0.1524" layer="91"/>
+<wire x1="-73.66" y1="30.48" x2="-83.82" y2="30.48" width="0.1524" layer="91"/>
+</segment>
+</net>

Commit message: forgot to connect a gnd pin
Connections:
- net N$3 renamed CH1
- net N$4 renamed CH2
- net N$6 renamed CH3
- net N$7 renamed CH4
- net N$8 renamed CH5
- net N$9 renamed CH6
- net GND: now also J5.SLEEVE
Changed lines of the file:
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@@
 <pinref part="JP2" gate="A" pin="3"/>
 <wire x1="12.7" y1="-111.76" x2="12.7" y2="-106.68" width="0.1524" layer="91"/>
-<wire x1="12.7" y1="-106.68" x2="-2.54" y2="-106.68" width="0.1524" layer="91"/>
+<wire x1="12.7" y1="-106.68" x2="5.08" y2="-106.68" width="0.1524" layer="91"/>
+<pinref part="J5" gate="G$1" pin="SLEEVE"/>
+<wire x1="5.08" y1="-106.68" x2="-2.54" y2="-106.68" width="0.1524" layer="91"/>
+<wire x1="5.08" y1="-116.84" x2="5.08" y2="-106.68" width="0.1524" layer="91"/>
+<junction x="5.08" y="-106.68"/>
 </segment>
 <segment>
@@
 </segment>
 </net>
-<net name="N$3" class="0">
+<net name="CH1" class="0">
 <segment>
 <pinref part="J1" gate="G$1" pin="TIP"/>
@@
 </segment>
 </net>
-<net name="N$4" class="0">
+<net name="CH2" class="0">
 <segment>
 <pinref part="R8" gate="G$1" pin="1"/>
@@
 </segment>
 </net>
-<net name="N$6" class="0">
+<net name="CH3" class="0">
 <segment>
 <pinref part="R9" gate="G$1" pin="1"/>
@@
 </segment>
 </net>
-<net name="N$7" class="0">
+<net name="CH4" class="0">
 <segment>
 <pinref part="R10" gate="G$1" pin="1"/>
@@
 </segment>
 </net>
-<net name="N$8" class="0">
+<net name="CH5" class="0">
 <segment>
 <pinref part="R11" gate="G$1" pin="1"/>
@@
 </segment>
 </net>
-<net name="N$9" class="0">
+<net name="CH6" class="0">
 <segment>
 <pinref part="R12" gate="G$1" pin="1"/>
