File: pcb/expansion/expansion.sch (EAGLE design)
At the start: 49 parts, among them IC3 STM32F042F4, J1 AUDIO_JACK_3.5MM_PTH, J2 AUDIO_JACK_3.5MM_PTH, J3 AUDIO_JACK_3.5MM_PTH, J4 AUDIO_JACK_3.5MM_PTH, J5 AUDIO_JACK_3.5MM_PTH, J6 AUDIO_JACK_3.5MM_PTH, SW3 324_SW, SW4 324_SW, U1 USBC_16P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

Commit message: updated silkscreen
Connections:
- net N$13: now also J1.RING
Changed lines of the file:
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@@
 <pinref part="JP7" gate="G$1" pin="1"/>
 <wire x1="-17.78" y1="27.94" x2="-27.94" y2="27.94" width="0.1524" layer="91"/>
+<pinref part="J1" gate="G$1" pin="RING"/>
+<wire x1="-33.02" y1="-111.76" x2="-33.02" y2="27.94" width="0.1524" layer="91"/>
+<wire x1="-33.02" y1="27.94" x2="-27.94" y2="27.94" width="0.1524" layer="91"/>
+<junction x="-27.94" y="27.94"/>
 </segment>
 </net>
