File: pcb/buzz/duckypad_buzz.brd (EAGLE design)
At the start: 109 x 96 mm, 161 parts, among them IC2 REG1117, Q1 BSS123, SW1 SPST_TACT-EVQQ2, SW2 SPST_TACT-EVQQ2, SW21 EC12E_SW, SW22 EC12E_SW, SW3 324_SW324_SWITCH_FOOT_HOLE, SW4 324_SW324_SWITCH_FOOT_HOLE, U1 USBC_16P, U2 USBC_16P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

Commit message: updated silkscreen
Parts:
- renumbered U$19 to U19, U$3 to BZ1
Changed lines of the file:
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@@
 <setting verticaltext="up"/>
 </settings>
-<grid distance="5" unitdist="mil" unit="mm" style="lines" multiple="1" display="yes" altdistance="1" altunitdist="mil" altunit="mil"/>
+<grid distance="5" unitdist="mil" unit="mil" style="lines" multiple="1" display="yes" altdistance="1" altunitdist="mil" altunit="mil"/>
 <layers>
 <layer number="1" name="Top" color="4" fill="1" visible="yes" active="yes"/>
-<layer number="2" name="pwr" color="49" fill="1" visible="yes" active="yes"/>
+<layer number="2" name="pwr" color="49" fill="1" visible="no" active="yes"/>
 <layer number="3" name="Route3" color="4" fill="3" visible="no" active="no"/>
 <layer number="4" name="Route4" color="1" fill="4" visible="no" active="no"/>
@@
 <layer number="13" name="Route13" color="4" fill="5" visible="no" active="no"/>
 <layer number="14" name="Route14" color="1" fill="6" visible="no" active="no"/>
-<layer number="15" name="gnd" color="23" fill="1" visible="yes" active="yes"/>
-<layer number="16" name="Bottom" color="1" fill="1" visible="yes" active="yes"/>
+<layer number="15" name="gnd" color="23" fill="1" visible="no" active="yes"/>
+<layer number="16" name="Bottom" color="1" fill="1" visible="no" active="yes"/>
 <layer number="17" name="Pads" color="2" fill="1" visible="yes" active="yes"/>
 <layer number="18" name="Vias" color="2" fill="1" visible="yes" active="yes"/>
 <layer number="19" name="Unrouted" color="6" fill="1" visible="yes" active="yes"/>
 <layer number="20" name="Dimension" color="15" fill="1" visible="yes" active="yes"/>
-<layer number="21" name="tPlace" color="7" fill="1" visible="no" active="yes"/>
+<layer number="21" name="tPlace" color="7" fill="1" visible="yes" active="yes"/>
 <layer number="22" name="bPlace" color="7" fill="1" visible="no" active="yes"/>
 <layer number="23" name="tOrigins" color="15" fill="1" visible="yes" active="yes"/>
-<layer number="24" name="bOrigins" color="15" fill="1" visible="yes" active="yes"/>
-<layer number="25" name="tNames" color="7" fill="1" visible="no" active="yes"/>
+<layer number="24" name="bOrigins" color="15" fill="1" visible="no" active="yes"/>
+<layer number="25" name="tNames" color="7" fill="1" visible="yes" active="yes"/>
 <layer number="26" name="bNames" color="7" fill="1" visible="no" active="yes"/>
 <layer number="27" name="tValues" color="7" fill="1" visible="no" active="yes"/>
@@
 <layer number="38" name="bTest" color="7" fill="1" visible="no" active="yes"/>
 <layer number="39" name="tKeepout" color="4" fill="11" visible="yes" active="yes"/>
-<layer number="40" name="bKeepout" color="1" fill="11" visible="yes" active="yes"/>
+<layer number="40" name="bKeepout" color="1" fill="11" visible="no" active="yes"/>
 <layer number="41" name="tRestrict" color="4" fill="10" visible="yes" active="yes"/>
-<layer number="42" name="bRestrict" color="1" fill="10" visible="yes" active="yes"/>
+<layer number="42" name="bRestrict" color="1" fill="10" visible="no" active="yes"/>
 <layer number="43" name="vRestrict" color="2" fill="10" visible="no" active="yes"/>
 <layer number="44" name="Drills" color="7" fill="1" visible="yes" active="yes"/>
@@
 <layer number="49" name="Reference" color="7" fill="1" visible="no" active="yes"/>
 <layer number="50" name="dxf" color="7" fill="1" visible="no" active="no"/>
-<layer number="51" name="tDocu" color="7" fill="1" visible="no" active="yes"/>
+<layer number="51" name="tDocu" color="7" fill="1" visible="yes" active="yes"/>
 <layer number="52" name="bDocu" color="7" fill="1" visible="no" active="yes"/>
 <layer number="53" name="tGND_GNDA" color="7" fill="9" visible="no" active="no"/>
@@
 </element>
 <element name="Y1" library="SparkFun-Clocks" package="CRYSTAL-SMD-3.2X2.5MM" value="16MHz_12pF" x="83.9224" y="61.9252" smashed="yes" rot="MR270">
+<attribute name="NAME" x="86.3354" y="63.0682" size="0.8128" layer="26" font="vector" rot="MR270" align="bottom-center"/>
 <attribute name="PROD_ID" value="XTAL-12454" x="84.9224" y="66.9252" size="1.778" layer="28" rot="MR270" display="off"/>
+<attribute name="VALUE" x="85.4464" y="61.9252" size="0.6096" layer="28" font="vector" ratio="20" rot="MR270" align="top-center"/>
 </element>
 <element name="R2" library="joyAnalog" package="0805" value="62K" x="88.027" y="71.948" smashed="yes" rot="MR180">
@@
 <attribute name="NAME" x="76.47" y="62.3545" size="0.8128" layer="26" rot="MR180"/>
 </element>
-<element name="U$19" library="SparkFun-Retired" package="SOT23-5" value="V_REG_TPS61040SMD" x="85.868" y="16.195" smashed="yes" rot="MR270"/>
+<element name="U19" library="SparkFun-Retired" package="SOT23-5" value="V_REG_TPS61040SMD" x="85.868" y="16.195" smashed="yes" rot="MR270">
+<attribute name="NAME" x="83.754" y="14.494" size="0.8128" layer="26" font="vector" rot="MR180"/>
+<attribute name="VALUE" x="86.0585" y="17.1475" size="0.4064" layer="28" rot="MR270"/>
+</element>
 <element name="C33" library="clock" package="0805" value="4.7uF" x="82.312" y="16.195" smashed="yes" rot="MR90">
 <attribute name="NAME" x="81.357" y="15.0495" size="0.8128" layer="26" rot="MR0"/>
@@
 <attribute name="NAME" x="94.3008" y="72.7329" size="0.8128" layer="26" rot="MR180"/>
 </element>
-<element name="L2" library="Discrete" package="L4030" value="4.7uH" x="83.963" y="20.066" smashed="yes" rot="MR180"/>
+<element name="L2" library="Discrete" package="L4030" value="4.7uH" x="83.963" y="20.066" smashed="yes" rot="MR180">
+<attribute name="NAME" x="82.058" y="23.368" size="0.8128" layer="26" ratio="10" rot="MR180"/>
+<attribute name="VALUE" x="81.931" y="23.241" size="0.8128" layer="28" ratio="10" rot="MR180"/>
+</element>
 <element name="C46" library="clock" package="0805" value="4.7uF" x="93.869" y="18.923" smashed="yes" rot="MR0">
 <attribute name="NAME" x="96.0915" y="20.193" size="0.8128" layer="26" rot="MR270"/>
@@
 <element name="JP1" library="SparkFun-Jumpers" package="SMT-JUMPER_2_NO_NO-SILK" value="JUMPER-SMT_2_NO_NO-SILK" x="79.613" y="95.25" smashed="yes" rot="MR0"/>
 <element name="JP4" library="SparkFun-Jumpers" package="SMT-JUMPER_2_NO_NO-SILK" value="JUMPER-SMT_2_NO_NO-SILK" x="108.2802" y="56.9976" smashed="yes" rot="R270"/>
-<element name="U$3" library="duckypad" package="BUZZ" value="BUZZ40402" x="107.061" y="2.667" smashed="yes" rot="MR0"/>
+<element name="BZ1" library="duckypad" package="BUZZ" value="BUZZ40402" x="107.061" y="2.667" smashed="yes" rot="MR0"/>
 <element name="Q1" library="transistor-small-signal" library_urn="urn:adsk.eagle:library:401" package="SOT23" package3d_urn="urn:adsk.eagle:package:28738/2" value="BSS123" x="96.266" y="6.477" smashed="yes" rot="MR270">
-<attribute name="NAME" x="94.869" y="4.826" size="1.27" layer="26" rot="MR180"/>
+<attribute name="NAME" x="95.377" y="9.017" size="0.8128" layer="26" rot="MR180"/>
 <attribute name="POPULARITY" value="21" x="100.457" y="6.477" size="1.778" layer="28" rot="MR270" display="off"/>
 <attribute name="VALUE" x="99.441" y="8.382" size="1.27" layer="28" rot="MR270"/>
@@
 <contactref element="C28" pad="1"/>
 <contactref element="C33" pad="1"/>
-<contactref element="U$19" pad="2"/>
+<contactref element="U19" pad="2"/>
 <contactref element="R10" pad="2"/>
 <contactref element="C31" pad="1"/>
@@
 <contactref element="C28" pad="2"/>
 <contactref element="C33" pad="2"/>
-<contactref element="U$19" pad="5"/>
-<contactref element="U$19" pad="4"/>
+<contactref element="U19" pad="5"/>
+<contactref element="U19" pad="4"/>
 <contactref element="U$2" pad="4"/>
 <contactref element="C36" pad="2"/>
@@
 <wire x1="83.566" y1="54.524" x2="84.421" y2="54.524" width="0.2032" layer="16"/>
 <wire x1="83.566" y1="54.124" x2="83.566" y2="54.524" width="0.2032" layer="16"/>
-<contactref element="U$3" pad="PLUS"/>
+<contactref element="BZ1" pad="PLUS"/>
 <contactref element="D22" pad="C"/>
 <via x="105.172" y="2.667" extent="1-16" drill="0.5"/>
@@
 </signal>
 <signal name="N$36">
-<contactref element="U$19" pad="1"/>
+<contactref element="U19" pad="1"/>
 <contactref element="L2" pad="2"/>
 <contactref element="D1" pad="A"/>
@@
 </signal>
 <signal name="N$39">
-<contactref element="U$19" pad="3"/>
+<contactref element="U19" pad="3"/>
 <contactref element="C35" pad="1"/>
 <contactref element="R10" pad="1"/>
@@
 </signal>
 <signal name="N$37">
-<contactref element="U$3" pad="MINUS"/>
+<contactref element="BZ1" pad="MINUS"/>
 <contactref element="Q1" pad="3"/>
 <contactref element="D22" pad="A"/>
