File: pcb/old/buzz_no_transistor/duckypad.brd (EAGLE design)
At the start: 109 x 96 mm, 161 parts, among them IC2 REG1117, Q1 BSS123, SW1 SPST_TACT-EVQQ2, SW2 SPST_TACT-EVQQ2, SW21 EC12E_SW, SW22 EC12E_SW, SW3 324_SW324_SWITCH_FOOT_HOLE, SW4 324_SW324_SWITCH_FOOT_HOLE, U1 USBC_16P, U19 V_REG_TPS61040SMD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

Commit message: updated pcb files
Parts:
- removed BZ1: BUZZ40402, duckypad:BUZZ
- removed D22: 1N4148, duckypad:ADAFRUIT_CHANGED_SOD-123
- removed Q1: BSS123, transistor-small-signal:SOT23
- added JP3: (no value), adafruit_changed:1X01-CLEANBIG
- added U$3: BUZZ40402, duckypad:BUZZ
- moved R19 1.25 mm to (100.5, 7.11), turned to 180 degrees
- renumbered U19 to U$19
Connections:
- net +3V3: no longer BZ1.PLUS, D22.C
- net GND: now also U$3.MINUS; no longer Q1.2, R19.1
- net N$37: now also R19.1, U$3.PLUS; no longer BZ1.MINUS, D22.A, Q1.3
- net N$70: no longer Q1.1
- net N$73: now also JP3.1
Routing:
- net +3V3: track 212.5 -> 190.0 mm, vias 33 -> 32
- net N$73: track 106.3 -> 122.6 mm, vias 2 -> 1
- net GND: track 70.6 -> 56.2 mm, vias 43 -> 42
- net N$37: track 11.4 -> 4.32 mm
- net N$70: track 78.2 -> 76.6 mm
- net N$72: track 106.9 -> 107.9 mm
Other:
- board text added: "duckyPad Pro dekuNukem R2 JAN2026"
- board text removed: "BZ1"
- board text removed: "duckyPad Pro dekuNukem JAN2026 R2"
