File: pcb/old/buzz_no_transistor/duckypad.sch (EAGLE design)
At the start: 161 parts, among them IC2 REG1117, Q1 BSS123, SW1 SPST_TACT-EVQQ2, SW2 SPST_TACT-EVQQ2, SW21 EC12E_SW, SW22 EC12E_SW, SW3 324_SW324_SWITCH_FOOT_HOLE, SW4 324_SW324_SWITCH_FOOT_HOLE, U1 USBC_16P, U19 V_REG_TPS61040SMD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

Commit message: updated pcb files
Parts:
- removed BZ1: BUZZ40402, duckypad:BUZZ40402
- removed D22: 1N4148, duckypad:ADAFRUIT_CHANGED_DIODESOD-123
- removed Q1: BSS123, transistor-small-signal:BSS123
- added JP3: (no value), adafruit_changed:PINHD-1X1CB
- added U$3: BUZZ40402, duckypad:BUZZ40402
- renumbered U19 to U$19
Connections:
- net +3V3: no longer BZ1.PLUS, D22.C
- net GND: now also U$3.MINUS; no longer Q1.S, R19.1
- net N$37: now also R19.1, U$3.PLUS; no longer BZ1.MINUS, D22.A, Q1.D
- net N$70: no longer Q1.G
- net N$73: now also JP3.1
Other:
- note removed: "BSS138"
- moved on the sheet: R19
Changed lines of the file:
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@@
 <drawing>
 <settings>
-<setting alwaysvectorfont="yes"/>
+<setting alwaysvectorfont="no"/>
 <setting keepoldvectorfont="yes"/>
 <setting verticaltext="up"/>
@@
 <part name="C28" library="clock" deviceset="CAP" device="0805" value="100nF"/>
 <part name="GND40" library="supply1" library_urn="urn:adsk.eagle:library:371" deviceset="GND" device=""/>
-<part name="U19" library="SparkFun-Retired" deviceset="V_REG_TPS61040" device="SMD"/>
+<part name="U$19" library="SparkFun-Retired" deviceset="V_REG_TPS61040" device="SMD"/>
 <part name="+3V32" library="supply1" library_urn="urn:adsk.eagle:library:371" deviceset="+3V3" device=""/>
 <part name="GND44" library="supply1" deviceset="GND" device=""/>
@@
 <part name="R17" library="joyAnalog" deviceset="RESISTOR" device="0805-RES" value="5K1"/>
 <part name="GND62" library="supply1" library_urn="urn:adsk.eagle:library:371" deviceset="GND" device=""/>
+<part name="JP3" library="adafruit_changed" deviceset="PINHD-1X1" device="CB"/>
 <part name="D1" library="duckypad" deviceset="ADAFRUIT_CHANGED_DIODE" device="SOD-123" value="1N4148"/>
 <part name="SW4" library="3pos_slide_switch" deviceset="324_SW" device="324_SWITCH_FOOT_HOLE" value="324_SW324_SWITCH_FOOT_HOLE"/>
@@
 <part name="GND65" library="supply1" deviceset="GND" device=""/>
 <part name="JP4" library="SparkFun-Jumpers" deviceset="JUMPER-SMT_2_NO" device="_NO-SILK"/>
-<part name="BZ1" library="duckypad" deviceset="BUZZ40402" device=""/>
-<part name="GND41" library="supply1" deviceset="GND" device=""/>
-<part name="Q1" library="transistor-small-signal" library_urn="urn:adsk.eagle:library:401" deviceset="BSS123" device="" package3d_urn="urn:adsk.eagle:package:28738/2"/>
-<part name="+3V2" library="supply1" library_urn="urn:adsk.eagle:library:371" deviceset="+3V3" device=""/>
-<part name="D22" library="duckypad" deviceset="ADAFRUIT_CHANGED_DIODE" device="SOD-123" value="1N4148"/>
+<part name="U$3" library="duckypad" deviceset="BUZZ40402" device=""/>
 <part name="R19" library="joyAnalog" deviceset="RESISTOR" device="0805-RES" value="5K1"/>
-<part name="GND67" library="supply1" deviceset="GND" device=""/>
+<part name="GND41" library="supply1" deviceset="GND" device=""/>
 </parts>
 <sheets>
@@
 <plain>
 <text x="297.18" y="-63.5" size="1.778" layer="94">40MHz!!!</text>
-<text x="63.5" y="-264.16" size="1.778" layer="94">BSS138</text>
 </plain>
 <instances>
@@
 <attribute name="VALUE" x="505.46" y="-35.56" size="1.778" layer="96"/>
 </instance>
-<instance part="U19" gate="G$1" x="190.5" y="-284.48" smashed="yes">
+<instance part="U$19" gate="G$1" x="190.5" y="-284.48" smashed="yes">
 <attribute name="NAME" x="185.42" y="-274.32" size="1.778" layer="95" rot="MR180"/>
 <attribute name="VALUE" x="185.42" y="-294.64" size="1.778" layer="96"/>
@@
 <attribute name="VALUE" x="373.38" y="-297.18" size="1.778" layer="96"/>
 </instance>
+<instance part="JP3" gate="G$1" x="317.5" y="-71.12" smashed="yes" rot="R180">
+<attribute name="NAME" x="323.85" y="-74.295" size="1.778" layer="95" rot="R180"/>
+<attribute name="VALUE" x="323.85" y="-66.04" size="1.778" layer="96" rot="R180"/>
+</instance>
 <instance part="D1" gate="G$1" x="210.82" y="-251.46" smashed="yes">
 <attribute name="NAME" x="208.28" y="-248.92" size="1.27" layer="95"/>
@@
 <attribute name="NAME" x="340.36" y="-7.62" size="1.778" layer="95" font="vector" rot="R90"/>
 </instance>
-<instance part="BZ1" gate="G$1" x="76.2" y="-228.6" smashed="yes" rot="MR270"/>
-<instance part="GND41" gate="1" x="76.2" y="-271.78" smashed="yes" rot="MR0">
-<attribute name="VALUE" x="78.74" y="-274.32" size="1.778" layer="96" rot="MR0"/>
-</instance>
-<instance part="Q1" gate="G$1" x="76.2" y="-256.54" smashed="yes" rot="MR0">
-<attribute name="NAME" x="73.66" y="-256.54" size="1.778" layer="95" rot="MR0"/>
-<attribute name="VALUE" x="73.66" y="-259.08" size="1.778" layer="96" rot="MR0"/>
-</instance>
-<instance part="+3V2" gate="G$1" x="76.2" y="-200.66" smashed="yes" rot="MR0">
-<attribute name="VALUE" x="78.74" y="-205.74" size="1.778" layer="96" rot="MR90"/>
-</instance>
-<instance part="D22" gate="G$1" x="60.96" y="-228.6" smashed="yes" rot="R90">
-<attribute name="NAME" x="58.42" y="-231.14" size="1.27" layer="95" rot="R90"/>
-<attribute name="VALUE" x="64.77" y="-231.14" size="1.27" layer="96" rot="R90"/>
-</instance>
-<instance part="R19" gate="G$1" x="91.44" y="-264.16" smashed="yes" rot="MR90">
-<attribute name="NAME" x="87.8586" y="-265.43" size="1.778" layer="95" rot="MR90"/>
-<attribute name="VALUE" x="85.598" y="-265.43" size="1.778" layer="96" rot="MR90"/>
+<instance part="U$3" gate="G$1" x="93.98" y="-220.98" smashed="yes" rot="MR0"/>
+<instance part="R19" gate="G$1" x="119.38" y="-220.98" smashed="yes" rot="MR180">
+<attribute name="NAME" x="118.11" y="-217.3986" size="1.778" layer="95" rot="MR180"/>
+<attribute name="VALUE" x="118.11" y="-215.138" size="1.778" layer="96" rot="MR180"/>
 </instance>
-<instance part="GND67" gate="1" x="91.44" y="-271.78" smashed="yes" rot="MR0">
-<attribute name="VALUE" x="93.98" y="-274.32" size="1.778" layer="96" rot="MR0"/>
+<instance part="GND41" gate="1" x="71.12" y="-223.52" smashed="yes" rot="MR0">
+<attribute name="VALUE" x="73.66" y="-226.06" size="1.778" layer="96" rot="MR0"/>
 </instance>
 </instances>
@@
 </segment>
 <segment>
-<pinref part="U19" gate="G$1" pin="GND"/>
+<pinref part="U$19" gate="G$1" pin="GND"/>
 <pinref part="GND45" gate="1" pin="GND"/>
 <wire x1="203.2" y1="-284.48" x2="205.74" y2="-284.48" width="0.1524" layer="91"/>
@@
 </segment>
 <segment>
-<pinref part="Q1" gate="G$1" pin="S"/>
 <pinref part="GND41" gate="1" pin="GND"/>
-<wire x1="76.2" y1="-269.24" x2="76.2" y2="-261.62" width="0.1524" layer="91"/>
-</segment>
-<segment>
-<pinref part="R19" gate="G$1" pin="1"/>
-<pinref part="GND67" gate="1" pin="GND"/>
+<pinref part="U$3" gate="G$1" pin="MINUS"/>
+<wire x1="71.12" y1="-220.98" x2="78.74" y2="-220.98" width="0.1524" layer="91"/>
 </segment>
 </net>
@@
 <wire x1="160.02" y1="-266.7" x2="172.72" y2="-266.7" width="0.1524" layer="91"/>
 <junction x="160.02" y="-266.7"/>
-<pinref part="U19" gate="G$1" pin="VIN"/>
+<pinref part="U$19" gate="G$1" pin="VIN"/>
 <wire x1="172.72" y1="-266.7" x2="182.88" y2="-266.7" width="0.1524" layer="91"/>
 <wire x1="180.34" y1="-279.4" x2="172.72" y2="-279.4" width="0.1524" layer="91"/>
 <wire x1="172.72" y1="-279.4" x2="172.72" y2="-266.7" width="0.1524" layer="91"/>
 <junction x="172.72" y="-266.7"/>
-<pinref part="U19" gate="G$1" pin="EN"/>
+<pinref part="U$19" gate="G$1" pin="EN"/>
 <wire x1="180.34" y1="-289.56" x2="172.72" y2="-289.56" width="0.1524" layer="91"/>
 <wire x1="172.72" y1="-289.56" x2="172.72" y2="-279.4" width="0.1524" layer="91"/>
@@
 <wire x1="147.32" y1="-208.28" x2="124.46" y2="-208.28" width="0.1524" layer="91"/>
 </segment>
-<segment>
-<pinref part="+3V2" gate="G$1" pin="+3V3"/>
-<pinref part="BZ1" gate="G$1" pin="PLUS"/>
-<wire x1="76.2" y1="-203.2" x2="76.2" y2="-213.36" width="0.1524" layer="91"/>
-<wire x1="76.2" y1="-213.36" x2="60.96" y2="-213.36" width="0.1524" layer="91"/>
-<wire x1="60.96" y1="-213.36" x2="60.96" y2="-226.06" width="0.1524" layer="91"/>
-<junction x="76.2" y="-213.36"/>
-<pinref part="D22" gate="G$1" pin="C"/>
-</segment>
 </net>
 <net name="USB_DP" class="0">
@@
 <segment>
 <wire x1="195.58" y1="-266.7" x2="205.74" y2="-266.7" width="0.1524" layer="91"/>
-<pinref part="U19" gate="G$1" pin="SW"/>
+<pinref part="U$19" gate="G$1" pin="SW"/>
 <wire x1="203.2" y1="-279.4" x2="205.74" y2="-279.4" width="0.1524" layer="91"/>
 <wire x1="205.74" y1="-279.4" x2="205.74" y2="-266.7" width="0.1524" layer="91"/>
@@
 <net name="N$39" class="0">
 <segment>
-<pinref part="U19" gate="G$1" pin="FB"/>
+<pinref part="U$19" gate="G$1" pin="FB"/>
 <wire x1="203.2" y1="-289.56" x2="208.28" y2="-289.56" width="0.1524" layer="91"/>
 <wire x1="208.28" y1="-289.56" x2="208.28" y2="-284.48" width="0.1524" layer="91"/>
@@
 <wire x1="373.38" y1="-220.98" x2="124.46" y2="-220.98" width="0.1524" layer="91"/>
 <pinref part="SH1" gate="G$1" pin="8"/>
-<pinref part="Q1" gate="G$1" pin="G"/>
-<wire x1="81.28" y1="-259.08" x2="91.44" y2="-259.08" width="0.1524" layer="91"/>
-<wire x1="91.44" y1="-259.08" x2="99.06" y2="-259.08" width="0.1524" layer="91"/>
-<wire x1="124.46" y1="-220.98" x2="99.06" y2="-220.98" width="0.1524" layer="91"/>
-<wire x1="99.06" y1="-220.98" x2="99.06" y2="-259.08" width="0.1524" layer="91"/>
-<junction x="124.46" y="-220.98"/>
 <pinref part="R19" gate="G$1" pin="2"/>
-<junction x="91.44" y="-259.08"/>
+<junction x="124.46" y="-220.98"/>
 </segment>
 </net>
@@
 <wire x1="347.98" y1="-71.12" x2="335.28" y2="-71.12" width="0.1524" layer="91"/>
 <wire x1="335.28" y1="-71.12" x2="335.28" y2="-226.06" width="0.1524" layer="91"/>
+<pinref part="JP3" gate="G$1" pin="1"/>
+<wire x1="335.28" y1="-71.12" x2="320.04" y2="-71.12" width="0.1524" layer="91"/>
+<junction x="335.28" y="-71.12"/>
 <wire x1="335.28" y1="-226.06" x2="124.46" y2="-226.06" width="0.1524" layer="91"/>
 <pinref part="SH1" gate="G$1" pin="10"/>
@@
 <net name="N$37" class="0">
 <segment>
-<pinref part="BZ1" gate="G$1" pin="MINUS"/>
-<pinref part="Q1" gate="G$1" pin="D"/>
-<wire x1="76.2" y1="-243.84" x2="76.2" y2="-251.46" width="0.1524" layer="91"/>
-<wire x1="76.2" y1="-243.84" x2="60.96" y2="-243.84" width="0.1524" layer="91"/>
-<wire x1="60.96" y1="-243.84" x2="60.96" y2="-231.14" width="0.1524" layer="91"/>
-<junction x="76.2" y="-243.84"/>
-<pinref part="D22" gate="G$1" pin="A"/>
+<pinref part="U$3" gate="G$1" pin="PLUS"/>
+<pinref part="R19" gate="G$1" pin="1"/>
+<wire x1="109.22" y1="-220.98" x2="114.3" y2="-220.98" width="0.1524" layer="91"/>
 </segment>
 </net>
